Commit message: materials.xacro

File: final_assemble_rover_description/urdf/materials.xacro (robot description, xacro)
@@ -4,3 +4,9 @@
   <color rgba="0.700 0.700 0.700 1.000"/>
 </material>
+<material name="red">
+  <color rgba="0.800 0.000 0.000 1.000"/>
+<material>
+<material name="black">
+  <color rgba="0.000 0.000 0.000 1.000"/>
+<material>
 </robot>

Commit message: materials

File: final_assemble_rover_description/urdf/materials.xacro (robot description, xacro)
@@ -6,7 +6,7 @@
 <material name="red">
   <color rgba="0.800 0.000 0.000 1.000"/>
-<material>
+</material>
 <material name="black">
   <color rgba="0.000 0.000 0.000 1.000"/>
-<material>
+</material>
 </robot>
