Commit message: link

File: final_assemble_rover_description/urdf/final_assemble_rover.xacro (robot description, xacro)
@@ -1,4 +1,10 @@
 <?xml version="1.0" ?>
 <robot name="final_assemble_rover" xmlns:xacro="http://www.ros.org/wiki/xacro">
+<link name="base_footprint"/>
+<joint name="base_footprint_joint" type="fixed">
+    <parent link="base_footprint"/>
+    <child link="base_link"/>
+    <origin xyz="0 0 0.1" rpy="0 -1.5708 0"/>
+</joint>
 <xacro:include filename="$(find final_assemble_rover_description)/urdf/materials.xacro" />
 <xacro:include filename="$(find final_assemble_rover_description)/urdf/final_assemble_rover.trans" />

Commit message: main_color

File: final_assemble_rover_description/urdf/final_assemble_rover.xacro (robot description, xacro)
@@ -21,5 +21,5 @@
       <mesh filename="package://final_assemble_rover_description/meshes/base_link.stl" scale="0.001 0.001 0.001"/>
     </geometry>
-    <material name="silver"/>
+    <material name="red"/>
   </visual>
   <collision>
@@ -101,5 +101,5 @@
       <mesh filename="package://final_assemble_rover_description/meshes/laser_link_1_1.stl" scale="0.001 0.001 0.001"/>
     </geometry>
-    <material name="silver"/>
+    <material name="black"/>
   </visual>
   <collision>

Commit message: rotate

File: final_assemble_rover_description/urdf/final_assemble_rover.xacro (robot description, xacro)
@@ -5,5 +5,5 @@
     <parent link="base_footprint"/>
     <child link="base_link"/>
-    <origin xyz="0 0 0.1" rpy="0 -1.5708 0"/>
+    <origin xyz="0 0 0.1" rpy="1.5708 0  0"/>
 </joint>
 <xacro:include filename="$(find final_assemble_rover_description)/urdf/materials.xacro" />

Commit message: final_rviz_setup

File: final_assemble_rover_description/urdf/final_assemble_rover.xacro (robot description, xacro)
@@ -101,5 +101,5 @@
       <mesh filename="package://final_assemble_rover_description/meshes/laser_link_1_1.stl" scale="0.001 0.001 0.001"/>
     </geometry>
-    <material name="black"/>
+    <material name="silver"/>
   </visual>
   <collision>

Commit message: inertia_fix

File: final_assemble_rover_description/urdf/final_assemble_rover.xacro (robot description, xacro)
@@ -14,6 +14,6 @@
   <inertial>
     <origin xyz="-0.012288395840692032 0.034460399576695354 0.0011969906215803167" rpy="0 0 0"/>
-    <mass value="0.7253853126312768"/>
-    <inertia ixx="0.000799" iyy="0.001019" izz="0.000579" ixy="2e-06" iyz="-3e-06" ixz="-1e-06"/>
+    <mass value="1.0"/>
+    <inertia ixx="0.01" ixy="0.0" ixz="0.0" iyy="0.01" iyz="0.0" izz="0.01" />
   </inertial>
   <visual>
@@ -34,6 +34,6 @@
   <inertial>
     <origin xyz="2.6630935998084304e-08 -2.8968758173167353e-07 0.009889971933162212" rpy="0 0 0"/>
-    <mass value="0.02765275799306101"/>
-    <inertia ixx="1.1e-05" iyy="1.1e-05" izz="1.9e-05" ixy="0.0" iyz="0.0" ixz="-0.0"/>
+    <mass value="1.0"/>
+    <inertia ixx="0.01" ixy="0.0" ixz="0.0" iyy="0.01" iyz="0.0" izz="0.01" />
   </inertial>
   <visual>
@@ -54,6 +54,6 @@
   <inertial>
     <origin xyz="-2.661230842117279e-07 7.953542884714393e-08 -0.009889974242528299" rpy="0 0 0"/>
-    <mass value="0.027652753131556615"/>
-    <inertia ixx="1.1e-05" iyy="1.1e-05" izz="1.9e-05" ixy="0.0" iyz="0.0" ixz="-0.0"/>
+    <mass value="1.0"/>
+    <inertia ixx="0.01" ixy="0.0" ixz="0.0" iyy="0.01" iyz="0.0" izz="0.01" />
   </inertial>
   <visual>
@@ -74,6 +74,6 @@
   <inertial>
     <origin xyz="4.5208840455945865e-07 -1.0408340855860843e-17 -6.181836115575344e-17" rpy="0 0 0"/>
-    <mass value="0.011278527065897603"/>
-    <inertia ixx="0.0" iyy="0.0" izz="0.0" ixy="-0.0" iyz="0.0" ixz="0.0"/>
+    <mass value="1.0"/>
+    <inertia ixx="0.01" ixy="0.0" ixz="0.0" iyy="0.01" iyz="0.0" izz="0.01" />
   </inertial>
   <visual>
@@ -94,6 +94,6 @@
   <inertial>
     <origin xyz="0.003060220670157498 0.024734911622924308 0.0005321423848153578" rpy="0 0 0"/>
-    <mass value="0.5737084736155983"/>
-    <inertia ixx="0.000249" iyy="0.000565" izz="0.000483" ixy="5.1e-05" iyz="-3e-06" ixz="5e-06"/>
+    <mass value="1.0"/>
+    <inertia ixx="0.01" ixy="0.0" ixz="0.0" iyy="0.01" iyz="0.0" izz="0.01" />
   </inertial>
   <visual>

Commit message: inertia

File: final_assemble_rover_description/urdf/final_assemble_rover.xacro (robot description, xacro)
@@ -1,10 +1,11 @@
 <?xml version="1.0" ?>
 <robot name="final_assemble_rover" xmlns:xacro="http://www.ros.org/wiki/xacro">
-<link name="base_footprint"/>
-<joint name="base_footprint_joint" type="fixed">
-    <parent link="base_footprint"/>
-    <child link="base_link"/>
-    <origin xyz="0 0 0.1" rpy="1.5708 0  0"/>
-</joint>
+<link name="base_footprint">
+    <inertial>
+        <mass value="0.0001"/>
+        <origin xyz="0 0 0" rpy="0 0 0"/>
+        <inertia ixx="0.0001" ixy="0.0" ixz="0.0" iyy="0.0001" iyz="0.0" izz="0.0001"/>
+    </inertial>
+</link>
 <xacro:include filename="$(find final_assemble_rover_description)/urdf/materials.xacro" />
 <xacro:include filename="$(find final_assemble_rover_description)/urdf/final_assemble_rover.trans" />

Commit message: update

File: final_assemble_rover_description/urdf/final_assemble_rover.xacro (robot description, xacro)
@@ -25,10 +25,4 @@
     <material name="red"/>
   </visual>
-  <collision>
-    <origin xyz="0 0 0" rpy="0 0 0"/>
-    <geometry>
-      <mesh filename="package://final_assemble_rover_description/meshes/base_link.stl" scale="0.001 0.001 0.001"/>
-    </geometry>
-  </collision>
 </link>
 <link name="right_wheel_link_1_1">
@@ -85,10 +79,4 @@
     <material name="silver"/>
   </visual>
-  <collision>
-    <origin xyz="-0.039746 0.0076 0.0" rpy="0 0 0"/>
-    <geometry>
-      <mesh filename="package://final_assemble_rover_description/meshes/castor_link_1_1.stl" scale="0.001 0.001 0.001"/>
-    </geometry>
-  </collision>
 </link>
 <link name="laser_link_1_1">
@@ -105,10 +93,4 @@
     <material name="silver"/>
   </visual>
-  <collision>
-    <origin xyz="0.0025 -0.09965 -0.0" rpy="0 0 0"/>
-    <geometry>
-      <mesh filename="package://final_assemble_rover_description/meshes/laser_link_1_1.stl" scale="0.001 0.001 0.001"/>
-    </geometry>
-  </collision>
 </link>
 <joint name="Revolute 19" type="continuous">

Commit message: update

File: final_assemble_rover_description/urdf/final_assemble_rover.xacro (robot description, xacro)
@@ -1,11 +1,18 @@
 <?xml version="1.0" ?>
 <robot name="final_assemble_rover" xmlns:xacro="http://www.ros.org/wiki/xacro">
-<link name="base_footprint">
-    <inertial>
-        <mass value="0.0001"/>
-        <origin xyz="0 0 0" rpy="0 0 0"/>
-        <inertia ixx="0.0001" ixy="0.0" ixz="0.0" iyy="0.0001" iyz="0.0" izz="0.0001"/>
-    </inertial>
-</link>
+<!-- The Root Link -->
+    <link name="base_footprint">
+        <inertial>
+            <mass value="0.0001"/>
+            <origin xyz="0 0 0" rpy="0 0 0"/>
+            <inertia ixx="0.0001" ixy="0.0" ixz="0.0" iyy="0.0001" iyz="0.0" izz="0.0001"/>
+        </inertial>
+    </link>
+    <!-- The Joint connecting the Root to the Chassis -->
+    <joint name="base_footprint_joint" type="fixed">
+        <parent link="base_footprint"/>
+        <child link="base_link"/>
+        <origin xyz="0 0 0.1" rpy="1.5708 0 0"/>
+    </joint>
 <xacro:include filename="$(find final_assemble_rover_description)/urdf/materials.xacro" />
 <xacro:include filename="$(find final_assemble_rover_description)/urdf/final_assemble_rover.trans" />

Commit message: update

File: final_assemble_rover_description/urdf/final_assemble_rover.xacro (robot description, xacro)
@@ -28,5 +28,5 @@
     <origin xyz="0 0 0" rpy="0 0 0"/>
     <geometry>
-      <mesh filename="package://final_assemble_rover_description/meshes/base_link.stl" scale="0.001 0.001 0.001"/>
+      <mesh filename="package://final_assemble_rover_description/meshes/base_link.stl" />
     </geometry>
     <material name="red"/>
@@ -42,5 +42,5 @@
     <origin xyz="0.029 -0.025 -0.06121" rpy="0 0 0"/>
     <geometry>
-      <mesh filename="package://final_assemble_rover_description/meshes/right_wheel_link_1_1.stl" scale="0.001 0.001 0.001"/>
+      <mesh filename="package://final_assemble_rover_description/meshes/right_wheel_link_1_1.stl" />
     </geometry>
     <material name="silver"/>
@@ -49,5 +49,5 @@
     <origin xyz="0.029 -0.025 -0.06121" rpy="0 0 0"/>
     <geometry>
-      <mesh filename="package://final_assemble_rover_description/meshes/right_wheel_link_1_1.stl" scale="0.001 0.001 0.001"/>
+      <mesh filename="package://final_assemble_rover_description/meshes/right_wheel_link_1_1.stl" />
     </geometry>
   </collision>
@@ -62,5 +62,5 @@
     <origin xyz="0.029 -0.025 0.06121" rpy="0 0 0"/>
     <geometry>
-      <mesh filename="package://final_assemble_rover_description/meshes/left_wheel_link_1_1.stl" scale="0.001 0.001 0.001"/>
+      <mesh filename="package://final_assemble_rover_description/meshes/left_wheel_link_1_1.stl" />
     </geometry>
     <material name="silver"/>
@@ -69,5 +69,5 @@
     <origin xyz="0.029 -0.025 0.06121" rpy="0 0 0"/>
     <geometry>
-      <mesh filename="package://final_assemble_rover_description/meshes/left_wheel_link_1_1.stl" scale="0.001 0.001 0.001"/>
+      <mesh filename="package://final_assemble_rover_description/meshes/left_wheel_link_1_1.stl" />
     </geometry>
   </collision>
@@ -82,5 +82,5 @@
     <origin xyz="-0.039746 0.0076 0.0" rpy="0 0 0"/>
     <geometry>
-      <mesh filename="package://final_assemble_rover_description/meshes/castor_link_1_1.stl" scale="0.001 0.001 0.001"/>
+      <mesh filename="package://final_assemble_rover_description/meshes/castor_link_1_1.stl"/>
     </geometry>
     <material name="silver"/>
@@ -96,5 +96,5 @@
     <origin xyz="0.0025 -0.09965 -0.0" rpy="0 0 0"/>
     <geometry>
-      <mesh filename="package://final_assemble_rover_description/meshes/laser_link_1_1.stl" scale="0.001 0.001 0.001"/>
+      <mesh filename="package://final_assemble_rover_description/meshes/laser_link_1_1.stl"/>
     </geometry>
     <material name="silver"/>

Commit message: final

File: final_assemble_rover_description/urdf/final_assemble_rover.xacro (robot description, xacro)
@@ -2,11 +2,5 @@
 <robot name="final_assemble_rover" xmlns:xacro="http://www.ros.org/wiki/xacro">
 <!-- The Root Link -->
-    <link name="base_footprint">
-        <inertial>
-            <mass value="0.0001"/>
-            <origin xyz="0 0 0" rpy="0 0 0"/>
-            <inertia ixx="0.0001" ixy="0.0" ixz="0.0" iyy="0.0001" iyz="0.0" izz="0.0001"/>
-        </inertial>
-    </link>
+    <link name="base_footprint"/>
     <!-- The Joint connecting the Root to the Chassis -->
     <joint name="base_footprint_joint" type="fixed">

Commit message: meshes

File: final_assemble_rover_description/urdf/final_assemble_rover.xacro (robot description, xacro)
@@ -22,5 +22,5 @@
     <origin xyz="0 0 0" rpy="0 0 0"/>
     <geometry>
-      <mesh filename="package://final_assemble_rover_description/meshes/base_link.stl" />
+      <mesh filename="file://$(find final_assemble_rover_description)/meshes/base_link.stl" />
     </geometry>
     <material name="red"/>

Commit message: meshes

File: final_assemble_rover_description/urdf/final_assemble_rover.xacro (robot description, xacro)
@@ -36,5 +36,5 @@
     <origin xyz="0.029 -0.025 -0.06121" rpy="0 0 0"/>
     <geometry>
-      <mesh filename="package://final_assemble_rover_description/meshes/right_wheel_link_1_1.stl" />
+      <mesh filename="file://$(find final_assemble_rover_description)/meshes/right_wheel_link_1_1.stl" />
     </geometry>
     <material name="silver"/>
@@ -43,5 +43,5 @@
     <origin xyz="0.029 -0.025 -0.06121" rpy="0 0 0"/>
     <geometry>
-      <mesh filename="package://final_assemble_rover_description/meshes/right_wheel_link_1_1.stl" />
+      <mesh filename="file://$(find final_assemble_rover_description)/meshes/right_wheel_link_1_1.stl" />
     </geometry>
   </collision>
@@ -56,5 +56,5 @@
     <origin xyz="0.029 -0.025 0.06121" rpy="0 0 0"/>
     <geometry>
-      <mesh filename="package://final_assemble_rover_description/meshes/left_wheel_link_1_1.stl" />
+      <mesh filename="file://$(find final_assemble_rover_description)/meshes/left_wheel_link_1_1.stl" />
     </geometry>
     <material name="silver"/>
@@ -63,5 +63,5 @@
     <origin xyz="0.029 -0.025 0.06121" rpy="0 0 0"/>
     <geometry>
-      <mesh filename="package://final_assemble_rover_description/meshes/left_wheel_link_1_1.stl" />
+      <mesh filename="file://$(find final_assemble_rover_description)/meshes/left_wheel_link_1_1.stl" />
     </geometry>
   </collision>
@@ -76,5 +76,5 @@
     <origin xyz="-0.039746 0.0076 0.0" rpy="0 0 0"/>
     <geometry>
-      <mesh filename="package://final_assemble_rover_description/meshes/castor_link_1_1.stl"/>
+      <mesh filename="file://$(find final_assemble_rover_description)/meshes/castor_link_1_1.stl"/>
     </geometry>
     <material name="silver"/>
@@ -90,5 +90,5 @@
     <origin xyz="0.0025 -0.09965 -0.0" rpy="0 0 0"/>
     <geometry>
-      <mesh filename="package://final_assemble_rover_description/meshes/laser_link_1_1.stl"/>
+      <mesh filename="file://$(find final_assemble_rover_description)/meshes/laser_link_1_1.stl"/>
     </geometry>
     <material name="silver"/>
