Commit message: xacro_update

File: final_assemble_rover_description/urdf/final_assemble_rover.xacro (robot description, xacro)
@@ -1,5 +1,5 @@
 <?xml version="1.0" ?>
 <robot name="final_assemble_rover" xmlns:xacro="http://www.ros.org/wiki/xacro">
-<!-- The Root Link -->
+    <!-- The Root Link -->
     <link name="base_footprint"/>
     <!-- The Joint connecting the Root to the Chassis -->
@@ -9,111 +9,129 @@
         <origin xyz="0 0 0.1" rpy="1.5708 0 0"/>
     </joint>
-<xacro:include filename="$(find final_assemble_rover_description)/urdf/materials.xacro" />
-<xacro:include filename="$(find final_assemble_rover_description)/urdf/final_assemble_rover.trans" />
-<xacro:include filename="$(find final_assemble_rover_description)/urdf/final_assemble_rover.gazebo" />
-<xacro:include filename="$(find final_assemble_rover_description)/urdf/gazebo_control.xacro" />
-<link name="base_link">
-  <inertial>
-    <origin xyz="-0.012288395840692032 0.034460399576695354 0.0011969906215803167" rpy="0 0 0"/>
-    <mass value="1.0"/>
-    <inertia ixx="0.01" ixy="0.0" ixz="0.0" iyy="0.01" iyz="0.0" izz="0.01" />
-  </inertial>
-  <visual>
-    <origin xyz="0 0 0" rpy="0 0 0"/>
-    <geometry>
-      <mesh filename="file://$(find final_assemble_rover_description)/meshes/base_link.stl" />
-    </geometry>
-    <material name="red"/>
-  </visual>
-</link>
-<link name="right_wheel_link_1_1">
-  <inertial>
-    <origin xyz="2.6630935998084304e-08 -2.8968758173167353e-07 0.009889971933162212" rpy="0 0 0"/>
-    <mass value="1.0"/>
-    <inertia ixx="0.01" ixy="0.0" ixz="0.0" iyy="0.01" iyz="0.0" izz="0.01" />
-  </inertial>
-  <visual>
-    <origin xyz="0.029 -0.025 -0.06121" rpy="0 0 0"/>
-    <geometry>
-      <mesh filename="file://$(find final_assemble_rover_description)/meshes/right_wheel_link_1_1.stl" />
-    </geometry>
-    <material name="silver"/>
-  </visual>
-  <collision>
-    <origin xyz="0.029 -0.025 -0.06121" rpy="0 0 0"/>
-    <geometry>
-      <mesh filename="file://$(find final_assemble_rover_description)/meshes/right_wheel_link_1_1.stl" />
-    </geometry>
-  </collision>
-</link>
-<link name="left_wheel_link_1_1">
-  <inertial>
-    <origin xyz="-2.661230842117279e-07 7.953542884714393e-08 -0.009889974242528299" rpy="0 0 0"/>
-    <mass value="1.0"/>
-    <inertia ixx="0.01" ixy="0.0" ixz="0.0" iyy="0.01" iyz="0.0" izz="0.01" />
-  </inertial>
-  <visual>
-    <origin xyz="0.029 -0.025 0.06121" rpy="0 0 0"/>
-    <geometry>
-      <mesh filename="file://$(find final_assemble_rover_description)/meshes/left_wheel_link_1_1.stl" />
-    </geometry>
-    <material name="silver"/>
-  </visual>
-  <collision>
-    <origin xyz="0.029 -0.025 0.06121" rpy="0 0 0"/>
-    <geometry>
-      <mesh filename="file://$(find final_assemble_rover_description)/meshes/left_wheel_link_1_1.stl" />
-    </geometry>
-  </collision>
-</link>
-<link name="castor_link_1_1">
-  <inertial>
-    <origin xyz="4.5208840455945865e-07 -1.0408340855860843e-17 -6.181836115575344e-17" rpy="0 0 0"/>
-    <mass value="1.0"/>
-    <inertia ixx="0.01" ixy="0.0" ixz="0.0" iyy="0.01" iyz="0.0" izz="0.01" />
-  </inertial>
-  <visual>
-    <origin xyz="-0.039746 0.0076 0.0" rpy="0 0 0"/>
-    <geometry>
-      <mesh filename="file://$(find final_assemble_rover_description)/meshes/castor_link_1_1.stl"/>
-    </geometry>
-    <material name="silver"/>
-  </visual>
-</link>
-<link name="laser_link_1_1">
-  <inertial>
-    <origin xyz="0.003060220670157498 0.024734911622924308 0.0005321423848153578" rpy="0 0 0"/>
-    <mass value="1.0"/>
-    <inertia ixx="0.01" ixy="0.0" ixz="0.0" iyy="0.01" iyz="0.0" izz="0.01" />
-  </inertial>
-  <visual>
-    <origin xyz="0.0025 -0.09965 -0.0" rpy="0 0 0"/>
-    <geometry>
-      <mesh filename="file://$(find final_assemble_rover_description)/meshes/laser_link_1_1.stl"/>
-    </geometry>
-    <material name="silver"/>
-  </visual>
-</link>
-<joint name="Revolute 19" type="continuous">
-  <origin xyz="-0.029 0.025 0.06121" rpy="0 0 0"/>
-  <parent link="base_link"/>
-  <child link="right_wheel_link_1_1"/>
-  <axis xyz="0.0 0.0 -1.0"/>
-</joint>
-<joint name="Revolute 20" type="continuous">
-  <origin xyz="-0.029 0.025 -0.06121" rpy="0 0 0"/>
-  <parent link="base_link"/>
-  <child link="left_wheel_link_1_1"/>
-  <axis xyz="0.0 0.0 -1.0"/>
-</joint>
-<joint name="Rigid 21" type="fixed">
-  <origin xyz="0.039746 -0.0076 0.0" rpy="0 0 0"/>
-  <parent link="base_link"/>
-  <child link="castor_link_1_1"/>
-</joint>
-<joint name="Rigid 22" type="fixed">
-  <origin xyz="-0.0025 0.09965 0.0" rpy="0 0 0"/>
-  <parent link="base_link"/>
-  <child link="laser_link_1_1"/>
-</joint>
+    <xacro:include filename="$(find final_assemble_rover_description)/urdf/materials.xacro" />
+    <xacro:include filename="$(find final_assemble_rover_description)/urdf/final_assemble_rover.trans" />
+    <xacro:include filename="$(find final_assemble_rover_description)/urdf/final_assemble_rover.gazebo" />
+    <xacro:include filename="$(find final_assemble_rover_description)/urdf/gazebo_control.xacro" />
+    <link name="base_link">
+        <inertial>
+            <origin xyz="-0.012288395840692032 0.034460399576695354 0.0011969906215803167" rpy="0 0 0"/>
+            <mass value="1.0"/>
+            <inertia ixx="0.01" ixy="0.0" ixz="0.0" iyy="0.01" iyz="0.0" izz="0.01" />
+        </inertial>
+        <visual>
+            <origin xyz="0 0 0" rpy="0 0 0"/>
+            <geometry>
+                <mesh filename="file://$(find final_assemble_rover_description)/meshes/base_link.stl" />
+            </geometry>
+            <material name="red"/>
+        </visual>
+        <collision>
+            <origin xyz="0 0 0" rpy="0 0 0"/>
+            <geometry>
+                <mesh filename="file://$(find final_assemble_rover_description)/meshes/base_link.stl" />
+            </geometry>
+        </collision>
+    </link>
+    <link name="right_wheel_link_1_1">
+        <inertial>
+            <origin xyz="2.6630935998084304e-08 -2.8968758173167353e-07 0.009889971933162212" rpy="0 0 0"/>
+            <mass value="1.0"/>
+            <inertia ixx="0.01" ixy="0.0" ixz="0.0" iyy="0.01" iyz="0.0" izz="0.01" />
+        </inertial>
+        <visual>
+            <origin xyz="0.029 -0.025 -0.06121" rpy="0 0 0"/>
+            <geometry>
+                <mesh filename="file://$(find final_assemble_rover_description)/meshes/right_wheel_link_1_1.stl" />
+            </geometry>
+            <material name="silver"/>
+        </visual>
+        <collision>
+            <origin xyz="0.029 -0.025 -0.06121" rpy="0 0 0"/>
+            <geometry>
+                <mesh filename="file://$(find final_assemble_rover_description)/meshes/right_wheel_link_1_1.stl" />
+            </geometry>
+        </collision>
+    </link>
+    <link name="left_wheel_link_1_1">
+        <inertial>
+            <origin xyz="-2.661230842117279e-07 7.953542884714393e-08 -0.009889974242528299" rpy="0 0 0"/>
+            <mass value="1.0"/>
+            <inertia ixx="0.01" ixy="0.0" ixz="0.0" iyy="0.01" iyz="0.0" izz="0.01" />
+        </inertial>
+        <visual>
+            <origin xyz="0.029 -0.025 0.06121" rpy="0 0 0"/>
+            <geometry>
+                <mesh filename="file://$(find final_assemble_rover_description)/meshes/left_wheel_link_1_1.stl" />
+            </geometry>
+            <material name="silver"/>
+        </visual>
+        <collision>
+            <origin xyz="0.029 -0.025 0.06121" rpy="0 0 0"/>
+            <geometry>
+                <mesh filename="file://$(find final_assemble_rover_description)/meshes/left_wheel_link_1_1.stl" />
+            </geometry>
+        </collision>
+    </link>
+    <link name="castor_link_1_1">
+        <inertial>
+            <origin xyz="4.5208840455945865e-07 -1.0408340855860843e-17 -6.181836115575344e-17" rpy="0 0 0"/>
+            <mass value="1.0"/>
+            <inertia ixx="0.01" ixy="0.0" ixz="0.0" iyy="0.01" iyz="0.0" izz="0.01" />
+        </inertial>
+        <visual>
+            <origin xyz="-0.039746 0.0076 0.0" rpy="0 0 0"/>
+            <geometry>
+                <mesh filename="file://$(find final_assemble_rover_description)/meshes/castor_link_1_1.stl"/>
+            </geometry>
+            <material name="silver"/>
+        </visual>
+        <collision>
+            <origin xyz="-0.039746 0.0076 0.0" rpy="0 0 0"/>
+            <geometry>
+                <mesh filename="file://$(find final_assemble_rover_description)/meshes/castor_link_1_1.stl"/>
+            </geometry>
+        </collision>
+    </link>
+    <link name="laser_link_1_1">
+        <inertial>
+            <origin xyz="0.003060220670157498 0.024734911622924308 0.0005321423848153578" rpy="0 0 0"/>
+            <mass value="1.0"/>
+            <inertia ixx="0.01" ixy="0.0" ixz="0.0" iyy="0.01" iyz="0.0" izz="0.01" />
+        </inertial>
+        <visual>
+            <origin xyz="0.0025 -0.09965 -0.0" rpy="0 0 0"/>
+            <geometry>
+                <mesh filename="file://$(find final_assemble_rover_description)/meshes/laser_link_1_1.stl"/>
+            </geometry>
+            <material name="silver"/>
+        </visual>
+        <collision>
+            <origin xyz="0.0025 -0.09965 -0.0" rpy="0 0 0"/>
+            <geometry>
+                <mesh filename="file://$(find final_assemble_rover_description)/meshes/laser_link_1_1.stl"/>
+            </geometry>
+        </collision>
+    </link>
+    <joint name="Revolute 19" type="continuous">
+        <origin xyz="-0.029 0.025 0.06121" rpy="0 0 0"/>
+        <parent link="base_link"/>
+        <child link="right_wheel_link_1_1"/>
+        <axis xyz="0.0 0.0 -1.0"/>
+    </joint>
+    <joint name="Revolute 20" type="continuous">
+        <origin xyz="-0.029 0.025 -0.06121" rpy="0 0 0"/>
+        <parent link="base_link"/>
+        <child link="left_wheel_link_1_1"/>
+        <axis xyz="0.0 0.0 -1.0"/>
+    </joint>
+    <joint name="Rigid 21" type="fixed">
+        <origin xyz="0.039746 -0.0076 0.0" rpy="0 0 0"/>
+        <parent link="base_link"/>
+        <child link="castor_link_1_1"/>
+    </joint>
+    <joint name="Rigid 22" type="fixed">
+        <origin xyz="-0.0025 0.09965 0.0" rpy="0 0 0"/>
+        <parent link="base_link"/>
+        <child link="laser_link_1_1"/>
+    </joint>
 </robot>

Commit message: inertia value

File: final_assemble_rover_description/urdf/final_assemble_rover.xacro (robot description, xacro)
@@ -36,6 +36,6 @@
         <inertial>
             <origin xyz="2.6630935998084304e-08 -2.8968758173167353e-07 0.009889971933162212" rpy="0 0 0"/>
-            <mass value="1.0"/>
-            <inertia ixx="0.01" ixy="0.0" ixz="0.0" iyy="0.01" iyz="0.0" izz="0.01" />
+            <mass value="0.1"/>
+<inertia ixx="0.001" ixy="0.0" ixz="0.0" iyy="0.001" iyz="0.0" izz="0.001" />
         </inertial>
         <visual>
@@ -56,6 +56,6 @@
         <inertial>
             <origin xyz="-2.661230842117279e-07 7.953542884714393e-08 -0.009889974242528299" rpy="0 0 0"/>
-            <mass value="1.0"/>
-            <inertia ixx="0.01" ixy="0.0" ixz="0.0" iyy="0.01" iyz="0.0" izz="0.01" />
+            <mass value="0.1"/>
+<inertia ixx="0.001" ixy="0.0" ixz="0.0" iyy="0.001" iyz="0.0" izz="0.001" />
         </inertial>
         <visual>

Commit message: update_inertial

File: final_assemble_rover_description/urdf/final_assemble_rover.xacro (robot description, xacro)
@@ -76,6 +76,6 @@
         <inertial>
             <origin xyz="4.5208840455945865e-07 -1.0408340855860843e-17 -6.181836115575344e-17" rpy="0 0 0"/>
-            <mass value="1.0"/>
-            <inertia ixx="0.01" ixy="0.0" ixz="0.0" iyy="0.01" iyz="0.0" izz="0.01" />
+            <mass value="0.01"/>
+<inertia ixx="0.0001" ixy="0.0" ixz="0.0" iyy="0.0001" iyz="0.0" izz="0.0001" />
         </inertial>
         <visual>
@@ -96,6 +96,6 @@
         <inertial>
             <origin xyz="0.003060220670157498 0.024734911622924308 0.0005321423848153578" rpy="0 0 0"/>
-            <mass value="1.0"/>
-            <inertia ixx="0.01" ixy="0.0" ixz="0.0" iyy="0.01" iyz="0.0" izz="0.01" />
+            <mass value="0.01"/>
+<inertia ixx="0.0001" ixy="0.0" ixz="0.0" iyy="0.0001" iyz="0.0" izz="0.0001" />
         </inertial>
         <visual>

Commit message: update_inertial

File: final_assemble_rover_description/urdf/final_assemble_rover.xacro (robot description, xacro)
@@ -26,10 +26,9 @@
             <material name="red"/>
         </visual>
-        <collision>
-            <origin xyz="0 0 0" rpy="0 0 0"/>
-            <geometry>
-                <mesh filename="file://$(find final_assemble_rover_description)/meshes/base_link.stl" />
-            </geometry>
-        </collision>
+<collision>
+  <origin xyz="0 0 0" rpy="0 0 0"/>
+  <geometry>
+    <box size="0.15 0.1 0.08"/> </geometry>
+</collision>
     </link>
     <link name="right_wheel_link_1_1">
@@ -46,10 +45,9 @@
             <material name="silver"/>
         </visual>
-        <collision>
-            <origin xyz="0.029 -0.025 -0.06121" rpy="0 0 0"/>
-            <geometry>
-                <mesh filename="file://$(find final_assemble_rover_description)/meshes/right_wheel_link_1_1.stl" />
-            </geometry>
-        </collision>
+<collision>
+  <origin xyz="0.029 -0.025 -0.06121" rpy="1.5708 0 0"/>
+  <geometry>
+    <cylinder radius="0.035" length="0.02"/> </geometry>
+</collision>
     </link>
     <link name="left_wheel_link_1_1">
@@ -66,10 +64,9 @@
             <material name="silver"/>
         </visual>
-        <collision>
-            <origin xyz="0.029 -0.025 0.06121" rpy="0 0 0"/>
-            <geometry>
-                <mesh filename="file://$(find final_assemble_rover_description)/meshes/left_wheel_link_1_1.stl" />
-            </geometry>
-        </collision>
+<collision>
+  <origin xyz="0.029 -0.025 -0.06121" rpy="1.5708 0 0"/>
+  <geometry>
+    <cylinder radius="0.035" length="0.02"/> </geometry>
+</collision>
     </link>
     <link name="castor_link_1_1">
@@ -86,10 +83,9 @@
             <material name="silver"/>
         </visual>
-        <collision>
-            <origin xyz="-0.039746 0.0076 0.0" rpy="0 0 0"/>
-            <geometry>
-                <mesh filename="file://$(find final_assemble_rover_description)/meshes/castor_link_1_1.stl"/>
-            </geometry>
-        </collision>
+<collision>
+  <origin xyz="0.029 -0.025 -0.06121" rpy="1.5708 0 0"/>
+  <geometry>
+    <cylinder radius="0.035" length="0.02"/> </geometry>
+</collision>
     </link>
     <link name="laser_link_1_1">
@@ -106,10 +102,9 @@
             <material name="silver"/>
         </visual>
-        <collision>
-            <origin xyz="0.0025 -0.09965 -0.0" rpy="0 0 0"/>
-            <geometry>
-                <mesh filename="file://$(find final_assemble_rover_description)/meshes/laser_link_1_1.stl"/>
-            </geometry>
-        </collision>
+<collision>
+  <origin xyz="0 0 0" rpy="0 0 0"/>
+  <geometry>
+    <box size="0.8 0.050 0.04"/> </geometry>
+</collision>
     </link>
     <joint name="Revolute 19" type="continuous">

Commit message: change

File: final_assemble_rover_description/urdf/final_assemble_rover.xacro (robot description, xacro)
@@ -46,7 +46,8 @@
         </visual>
 <collision>
-  <origin xyz="0.029 -0.025 -0.06121" rpy="1.5708 0 0"/>
+  <origin xyz="0.029 -0.025 -0.06121" rpy="0 0 0"/>
   <geometry>
-    <cylinder radius="0.035" length="0.02"/> </geometry>
+    <cylinder radius="0.035" length="0.02"/>
+  </geometry>
 </collision>
     </link>

Commit message: psh

File: final_assemble_rover_description/urdf/final_assemble_rover.xacro (robot description, xacro)
@@ -66,7 +66,8 @@
         </visual>
 <collision>
-  <origin xyz="0.029 -0.025 -0.06121" rpy="1.5708 0 0"/>
+  <origin xyz="0.029 -0.025 0.06121" rpy="0 0 0"/>
   <geometry>
-    <cylinder radius="0.035" length="0.02"/> </geometry>
+    <cylinder radius="0.035" length="0.02"/>
+  </geometry>
 </collision>
     </link>

Commit message: inert fix

File: final_assemble_rover_description/urdf/final_assemble_rover.xacro (robot description, xacro)
@@ -46,5 +46,5 @@
         </visual>
 <collision>
-  <origin xyz="0.029 -0.025 -0.06121" rpy="0 0 0"/>
+  <origin xyz="0 0 0" rpy="0 0 0"/>
   <geometry>
     <cylinder radius="0.035" length="0.02"/>
@@ -66,5 +66,5 @@
         </visual>
 <collision>
-  <origin xyz="0.029 -0.025 0.06121" rpy="0 0 0"/>
+  <origin xyz="0 0 0" rpy="0 0 0"/>
   <geometry>
     <cylinder radius="0.035" length="0.02"/>
@@ -86,5 +86,5 @@
         </visual>
 <collision>
-  <origin xyz="0.029 -0.025 -0.06121" rpy="1.5708 0 0"/>
+  <origin xyz="0 0 0" rpy="1.5708 0 0"/>
   <geometry>
     <cylinder radius="0.035" length="0.02"/> </geometry>

Commit message: temp_fix

File: final_assemble_rover_description/urdf/final_assemble_rover.xacro (robot description, xacro)
@@ -46,5 +46,5 @@
         </visual>
 <collision>
-  <origin xyz="0 0 0" rpy="0 0 0"/>
+  <origin xyz="0.029 -0.025 -0.06121" rpy="0 0 0"/>
   <geometry>
     <cylinder radius="0.035" length="0.02"/>
@@ -66,5 +66,5 @@
         </visual>
 <collision>
-  <origin xyz="0 0 0" rpy="0 0 0"/>
+  <origin xyz="0.029 -0.025 0.06121" rpy="0 0 0"/>
   <geometry>
     <cylinder radius="0.035" length="0.02"/>
@@ -86,5 +86,5 @@
         </visual>
 <collision>
-  <origin xyz="0 0 0" rpy="1.5708 0 0"/>
+  <origin xyz="0.029 -0.025 -0.06121" rpy="1.5708 0 0"/>
   <geometry>
     <cylinder radius="0.035" length="0.02"/> </geometry>
@@ -111,5 +111,5 @@
     </link>
     <joint name="Revolute 19" type="continuous">
-        <origin xyz="-0.029 0.025 0.06121" rpy="0 0 0"/>
+        <origin xyz="0 0 0" rpy="0 0 0"/>
         <parent link="base_link"/>
         <child link="right_wheel_link_1_1"/>
@@ -117,5 +117,5 @@
     </joint>
     <joint name="Revolute 20" type="continuous">
-        <origin xyz="-0.029 0.025 -0.06121" rpy="0 0 0"/>
+        <origin xyz="0 0 0" rpy="0 0 0"/>
         <parent link="base_link"/>
         <child link="left_wheel_link_1_1"/>
