Commit message: revert

File: final_assemble_rover_description/urdf/final_assemble_rover.xacro (robot description, xacro)
@@ -1,4 +1,8 @@
 <?xml version="1.0" ?>
 <robot name="final_assemble_rover" xmlns:xacro="http://www.ros.org/wiki/xacro">
+    <xacro:include filename="$(find final_assemble_rover_description)/urdf/materials.xacro" />
+    <xacro:include filename="$(find final_assemble_rover_description)/urdf/final_assemble_rover.trans" />
+    <xacro:include filename="$(find final_assemble_rover_description)/urdf/final_assemble_rover.gazebo" />
+    <xacro:include filename="$(find final_assemble_rover_description)/urdf/gazebo_control.xacro" />
     <!-- ROOT LINK -->
     <link name="base_footprint"/>
@@ -6,14 +10,9 @@
         <parent link="base_footprint"/>
         <child link="base_link"/>
-        <origin xyz="0 0 0.1" rpy="1.5708 0 0"/>
+        <origin xyz="0 0 0.1" rpy="0 0 0"/>
     </joint>
-    <xacro:include filename="$(find final_assemble_rover_description)/urdf/materials.xacro" />
-    <xacro:include filename="$(find final_assemble_rover_description)/urdf/final_assemble_rover.trans" />
-    <xacro:include filename="$(find final_assemble_rover_description)/urdf/final_assemble_rover.gazebo" />
-    <xacro:include filename="$(find final_assemble_rover_description)/urdf/gazebo_control.xacro" />
     <!-- CHASSIS -->
     <link name="base_link">
         <inertial>
-            <!-- ZEROED CENTER OF MASS SO IT DOESN'T TIP -->
             <origin xyz="0 0 0" rpy="0 0 0"/>
             <mass value="1.0"/>
@@ -22,15 +21,10 @@
         <visual>
             <origin xyz="0 0 0" rpy="0 0 0"/>
-            <geometry>
-                <mesh filename="file://$(find final_assemble_rover_description)/meshes/base_link.stl" />
-            </geometry>
+            <geometry><box size="0.2 0.15 0.08"/></geometry>
             <material name="red"/>
         </visual>
-        <!-- BELLY FIX: Shifted up and shrunk so it can't touch the floor -->
         <collision>
-            <origin xyz="0 0.05 0" rpy="0 0 0"/>
-            <geometry>
-                <box size="0.1 0.05 0.08"/>
-            </geometry>
+            <origin xyz="0 0 0" rpy="0 0 0"/>
+            <geometry><box size="0.2 0.15 0.08"/></geometry>
         </collision>
     </link>
@@ -43,24 +37,18 @@
         </inertial>
         <visual>
-            <!-- EXACT ORIGINAL FUSION OFFSET -->
-            <origin xyz="0.029 -0.025 -0.06121" rpy="0 0 0"/>
-            <geometry>
-                <mesh filename="file://$(find final_assemble_rover_description)/meshes/right_wheel_link_1_1.stl" />
-            </geometry>
+            <origin xyz="0 0 0" rpy="1.5708 0 0"/>
+            <geometry><cylinder radius="0.04" length="0.02"/></geometry>
             <material name="silver"/>
         </visual>
         <collision>
-            <origin xyz="0 0 0" rpy="0 0 0"/>
-            <geometry>
-                <cylinder radius="0.035" length="0.02"/>
-            </geometry>
+            <origin xyz="0 0 0" rpy="1.5708 0 0"/>
+            <geometry><cylinder radius="0.04" length="0.02"/></geometry>
         </collision>
     </link>
-    <joint name="Revolute 19" type="continuous">
-        <!-- EXACT ORIGINAL JOINT OFFSET -->
-        <origin xyz="-0.029 0.025 0.06121" rpy="0 0 0"/>
+    <joint name="Revolute_19" type="continuous">
+        <origin xyz="-0.05 -0.09 -0.04" rpy="0 0 0"/>
         <parent link="base_link"/>
         <child link="right_wheel_link_1_1"/>
-        <axis xyz="0.0 0.0 -1.0"/>
+        <axis xyz="0 1 0"/>
     </joint>
     <!-- LEFT WHEEL -->
@@ -72,24 +60,18 @@
         </inertial>
         <visual>
-            <!-- EXACT ORIGINAL FUSION OFFSET -->
-            <origin xyz="0.029 -0.025 0.06121" rpy="0 0 0"/>
-            <geometry>
-                <mesh filename="file://$(find final_assemble_rover_description)/meshes/left_wheel_link_1_1.stl" />
-            </geometry>
+            <origin xyz="0 0 0" rpy="1.5708 0 0"/>
+            <geometry><cylinder radius="0.04" length="0.02"/></geometry>
             <material name="silver"/>
         </visual>
         <collision>
-            <origin xyz="0 0 0" rpy="0 0 0"/>
-            <geometry>
-                <cylinder radius="0.035" length="0.02"/>
-            </geometry>
+            <origin xyz="0 0 0" rpy="1.5708 0 0"/>
+            <geometry><cylinder radius="0.04" length="0.02"/></geometry>
         </collision>
     </link>
-    <joint name="Revolute 20" type="continuous">
-        <!-- EXACT ORIGINAL JOINT OFFSET -->
-        <origin xyz="-0.029 0.025 -0.06121" rpy="0 0 0"/>
+    <joint name="Revolute_20" type="continuous">
+        <origin xyz="-0.05 0.09 -0.04" rpy="0 0 0"/>
         <parent link="base_link"/>
         <child link="left_wheel_link_1_1"/>
-        <axis xyz="0.0 0.0 -1.0"/>
+        <axis xyz="0 1 0"/>
     </joint>
     <!-- CASTOR WHEEL -->
@@ -101,22 +83,15 @@
         </inertial>
         <visual>
-            <!-- EXACT ORIGINAL FUSION OFFSET -->
-            <origin xyz="-0.039746 0.0076 0.0" rpy="0 0 0"/>
-            <geometry>
-                <mesh filename="file://$(find final_assemble_rover_description)/meshes/castor_link_1_1.stl"/>
-            </geometry>
+            <origin xyz="0 0 0" rpy="0 0 0"/>
+            <geometry><sphere radius="0.02"/></geometry>
             <material name="silver"/>
         </visual>
         <collision>
             <origin xyz="0 0 0" rpy="0 0 0"/>
-            <geometry>
-                <!-- TINY RADIUS SO IT DOESN'T JACK UP THE ROVER -->
-                <sphere radius="0.002"/>
-            </geometry>
+            <geometry><sphere radius="0.02"/></geometry>
         </collision>
     </link>
-    <joint name="Rigid 21" type="fixed">
-        <!-- EXACT ORIGINAL JOINT OFFSET -->
-        <origin xyz="0.039746 -0.0076 0.0" rpy="0 0 0"/>
+    <joint name="Rigid_21" type="fixed">
+        <origin xyz="0.08 0 -0.06" rpy="0 0 0"/>
         <parent link="base_link"/>
         <child link="castor_link_1_1"/>
@@ -130,20 +105,15 @@
         </inertial>
         <visual>
-            <!-- EXACT ORIGINAL FUSION OFFSET -->
-            <origin xyz="0.0025 -0.09965 -0.0" rpy="0 0 0"/>
-            <geometry>
-                <mesh filename="file://$(find final_assemble_rover_description)/meshes/laser_link_1_1.stl"/>
-            </geometry>
+            <origin xyz="0 0 0" rpy="0 0 0"/>
+            <geometry><box size="0.03 0.03 0.03"/></geometry>
             <material name="silver"/>
         </visual>
         <collision>
             <origin xyz="0 0 0" rpy="0 0 0"/>
-            <geometry>
-                <box size="0.03 0.03 0.03"/>
-            </geometry>
+            <geometry><box size="0.03 0.03 0.03"/></geometry>
         </collision>
     </link>
-    <joint name="Rigid 22" type="fixed">
-        <origin xyz="-0.0025 0.09965 0.0" rpy="0 0 0"/>
+    <joint name="Rigid_22" type="fixed">
+        <origin xyz="0.05 0 0.05" rpy="0 0 0"/>
         <parent link="base_link"/>
         <child link="laser_link_1_1"/>

Commit message: update_xacro_rover'

File: final_assemble_rover_description/urdf/final_assemble_rover.xacro (robot description, xacro)
@@ -20,6 +20,7 @@
         </inertial>
         <visual>
-            <origin xyz="0 0 0" rpy="0 0 0"/>
-            <geometry><box size="0.2 0.15 0.08"/></geometry>
+            <!-- 90 degree pitch maps Fusion Z-up to ROS standard -->
+            <origin xyz="0 0 0" rpy="1.5708 0 0"/>
+            <geometry><mesh filename="file://$(find final_assemble_rover_description)/meshes/base_link.stl" /></geometry>
             <material name="red"/>
         </visual>
@@ -38,5 +39,5 @@
         <visual>
             <origin xyz="0 0 0" rpy="1.5708 0 0"/>
-            <geometry><cylinder radius="0.04" length="0.02"/></geometry>
+            <geometry><mesh filename="file://$(find final_assemble_rover_description)/meshes/right_wheel_link_1.stl" /></geometry>
             <material name="silver"/>
         </visual>
@@ -46,5 +47,5 @@
         </collision>
     </link>
-    <joint name="Revolute_19" type="continuous">
+    <joint name="Revolute 19" type="continuous">
         <origin xyz="-0.05 -0.09 -0.04" rpy="0 0 0"/>
         <parent link="base_link"/>
@@ -61,5 +62,5 @@
         <visual>
             <origin xyz="0 0 0" rpy="1.5708 0 0"/>
-            <geometry><cylinder radius="0.04" length="0.02"/></geometry>
+            <geometry><mesh filename="file://$(find final_assemble_rover_description)/meshes/left_wheel_link_1.stl" /></geometry>
             <material name="silver"/>
         </visual>
@@ -69,5 +70,5 @@
         </collision>
     </link>
-    <joint name="Revolute_20" type="continuous">
+    <joint name="Revolute 20" type="continuous">
         <origin xyz="-0.05 0.09 -0.04" rpy="0 0 0"/>
         <parent link="base_link"/>
@@ -83,6 +84,6 @@
         </inertial>
         <visual>
-            <origin xyz="0 0 0" rpy="0 0 0"/>
-            <geometry><sphere radius="0.02"/></geometry>
+            <origin xyz="0 0 0" rpy="1.5708 0 0"/>
+            <geometry><mesh filename="file://$(find final_assemble_rover_description)/meshes/castor_link_1.stl"/></geometry>
             <material name="silver"/>
         </visual>
@@ -92,5 +93,5 @@
         </collision>
     </link>
-    <joint name="Rigid_21" type="fixed">
+    <joint name="Rigid 21" type="fixed">
         <origin xyz="0.08 0 -0.06" rpy="0 0 0"/>
         <parent link="base_link"/>
@@ -105,6 +106,6 @@
         </inertial>
         <visual>
-            <origin xyz="0 0 0" rpy="0 0 0"/>
-            <geometry><box size="0.03 0.03 0.03"/></geometry>
+            <origin xyz="0 0 0" rpy="1.5708 0 0"/>
+            <geometry><mesh filename="file://$(find final_assemble_rover_description)/meshes/laser_link_1.stl"/></geometry>
             <material name="silver"/>
         </visual>
@@ -114,5 +115,5 @@
         </collision>
     </link>
-    <joint name="Rigid_22" type="fixed">
+    <joint name="Rigid 22" type="fixed">
         <origin xyz="0.05 0 0.05" rpy="0 0 0"/>
         <parent link="base_link"/>

Commit message: update_check

File: final_assemble_rover_description/urdf/final_assemble_rover.xacro (robot description, xacro)
@@ -5,12 +5,11 @@
     <xacro:include filename="$(find final_assemble_rover_description)/urdf/final_assemble_rover.gazebo" />
     <xacro:include filename="$(find final_assemble_rover_description)/urdf/gazebo_control.xacro" />
-    <!-- ROOT LINK -->
+    <!-- ORIGINAL 90-DEGREE PITCH -->
     <link name="base_footprint"/>
     <joint name="base_footprint_joint" type="fixed">
         <parent link="base_footprint"/>
         <child link="base_link"/>
-        <origin xyz="0 0 0.1" rpy="0 0 0"/>
+        <origin xyz="0 0 0.1" rpy="1.5708 0 0"/>
     </joint>
-    <!-- CHASSIS -->
     <link name="base_link">
         <inertial>
@@ -20,15 +19,18 @@
         </inertial>
         <visual>
-            <!-- 90 degree pitch maps Fusion Z-up to ROS standard -->
-            <origin xyz="0 0 0" rpy="1.5708 0 0"/>
-            <geometry><mesh filename="file://$(find final_assemble_rover_description)/meshes/base_link.stl" /></geometry>
+            <origin xyz="0 0 0" rpy="0 0 0"/>
+            <geometry>
+                <mesh filename="file://$(find final_assemble_rover_description)/meshes/base_link.stl" />
+            </geometry>
             <material name="red"/>
         </visual>
+        <!-- Elevated collision box so the belly doesn't scrape -->
         <collision>
-            <origin xyz="0 0 0" rpy="0 0 0"/>
-            <geometry><box size="0.2 0.15 0.08"/></geometry>
+            <origin xyz="0 0.05 0" rpy="0 0 0"/>
+            <geometry>
+                <box size="0.1 0.05 0.08"/>
+            </geometry>
         </collision>
     </link>
-    <!-- RIGHT WHEEL -->
     <link name="right_wheel_link_1_1">
         <inertial>
@@ -38,20 +40,24 @@
         </inertial>
         <visual>
-            <origin xyz="0 0 0" rpy="1.5708 0 0"/>
-            <geometry><mesh filename="file://$(find final_assemble_rover_description)/meshes/right_wheel_link_1.stl" /></geometry>
+            <!-- ORIGINAL OFFSET TO PUSH IT BACK TO THE SIDE -->
+            <origin xyz="0.029 -0.025 -0.06121" rpy="0 0 0"/>
+            <geometry>
+                <mesh filename="file://$(find final_assemble_rover_description)/meshes/right_wheel_link_1.stl" />
+            </geometry>
             <material name="silver"/>
         </visual>
         <collision>
-            <origin xyz="0 0 0" rpy="1.5708 0 0"/>
-            <geometry><cylinder radius="0.04" length="0.02"/></geometry>
+            <origin xyz="0 0 0" rpy="0 0 0"/>
+            <geometry>
+                <cylinder radius="0.035" length="0.02"/>
+            </geometry>
         </collision>
     </link>
     <joint name="Revolute 19" type="continuous">
-        <origin xyz="-0.05 -0.09 -0.04" rpy="0 0 0"/>
+        <origin xyz="-0.029 0.025 0.06121" rpy="0 0 0"/>
         <parent link="base_link"/>
         <child link="right_wheel_link_1_1"/>
-        <axis xyz="0 1 0"/>
+        <axis xyz="0.0 0.0 -1.0"/>
     </joint>
-    <!-- LEFT WHEEL -->
     <link name="left_wheel_link_1_1">
         <inertial>
@@ -61,20 +67,24 @@
         </inertial>
         <visual>
-            <origin xyz="0 0 0" rpy="1.5708 0 0"/>
-            <geometry><mesh filename="file://$(find final_assemble_rover_description)/meshes/left_wheel_link_1.stl" /></geometry>
+            <!-- ORIGINAL OFFSET TO PUSH IT BACK TO THE SIDE -->
+            <origin xyz="0.029 -0.025 0.06121" rpy="0 0 0"/>
+            <geometry>
+                <mesh filename="file://$(find final_assemble_rover_description)/meshes/left_wheel_link_1.stl" />
+            </geometry>
             <material name="silver"/>
         </visual>
         <collision>
-            <origin xyz="0 0 0" rpy="1.5708 0 0"/>
-            <geometry><cylinder radius="0.04" length="0.02"/></geometry>
+            <origin xyz="0 0 0" rpy="0 0 0"/>
+            <geometry>
+                <cylinder radius="0.035" length="0.02"/>
+            </geometry>
         </collision>
     </link>
     <joint name="Revolute 20" type="continuous">
-        <origin xyz="-0.05 0.09 -0.04" rpy="0 0 0"/>
+        <origin xyz="-0.029 0.025 -0.06121" rpy="0 0 0"/>
         <parent link="base_link"/>
         <child link="left_wheel_link_1_1"/>
-        <axis xyz="0 1 0"/>
+        <axis xyz="0.0 0.0 -1.0"/>
     </joint>
-    <!-- CASTOR WHEEL -->
     <link name="castor_link_1_1">
         <inertial>
@@ -84,19 +94,22 @@
         </inertial>
         <visual>
-            <origin xyz="0 0 0" rpy="1.5708 0 0"/>
-            <geometry><mesh filename="file://$(find final_assemble_rover_description)/meshes/castor_link_1.stl"/></geometry>
+            <origin xyz="-0.039746 0.0076 0.0" rpy="0 0 0"/>
+            <geometry>
+                <mesh filename="file://$(find final_assemble_rover_description)/meshes/castor_link_1.stl"/>
+            </geometry>
             <material name="silver"/>
         </visual>
         <collision>
             <origin xyz="0 0 0" rpy="0 0 0"/>
-            <geometry><sphere radius="0.02"/></geometry>
+            <geometry>
+                <sphere radius="0.002"/>
+            </geometry>
         </collision>
     </link>
     <joint name="Rigid 21" type="fixed">
-        <origin xyz="0.08 0 -0.06" rpy="0 0 0"/>
+        <origin xyz="0.039746 -0.0076 0.0" rpy="0 0 0"/>
         <parent link="base_link"/>
         <child link="castor_link_1_1"/>
     </joint>
-    <!-- LASER SENSOR -->
     <link name="laser_link_1_1">
         <inertial>
@@ -106,15 +119,19 @@
         </inertial>
         <visual>
-            <origin xyz="0 0 0" rpy="1.5708 0 0"/>
-            <geometry><mesh filename="file://$(find final_assemble_rover_description)/meshes/laser_link_1.stl"/></geometry>
+            <origin xyz="0.0025 -0.09965 -0.0" rpy="0 0 0"/>
+            <geometry>
+                <mesh filename="file://$(find final_assemble_rover_description)/meshes/laser_link_1.stl"/>
+            </geometry>
             <material name="silver"/>
         </visual>
         <collision>
             <origin xyz="0 0 0" rpy="0 0 0"/>
-            <geometry><box size="0.03 0.03 0.03"/></geometry>
+            <geometry>
+                <box size="0.03 0.03 0.03"/>
+            </geometry>
         </collision>
     </link>
     <joint name="Rigid 22" type="fixed">
-        <origin xyz="0.05 0 0.05" rpy="0 0 0"/>
+        <origin xyz="-0.0025 0.09965 0.0" rpy="0 0 0"/>
         <parent link="base_link"/>
         <child link="laser_link_1_1"/>
