Commit message: stl push

File: final_assemble_rover_description/urdf/final_assemble_rover.xacro (robot description, xacro)
@@ -1,139 +1,6509 @@
 <?xml version="1.0" ?>
-<robot name="final_assemble_rover" xmlns:xacro="http://www.ros.org/wiki/xacro">
-    <xacro:include filename="$(find final_assemble_rover_description)/urdf/materials.xacro" />
-    <xacro:include filename="$(find final_assemble_rover_description)/urdf/final_assemble_rover.trans" />
-    <xacro:include filename="$(find final_assemble_rover_description)/urdf/final_assemble_rover.gazebo" />
-    <xacro:include filename="$(find final_assemble_rover_description)/urdf/gazebo_control.xacro" />
-    <!-- ORIGINAL 90-DEGREE PITCH -->
-    <link name="base_footprint"/>
-    <joint name="base_footprint_joint" type="fixed">
-        <parent link="base_footprint"/>
-        <child link="base_link"/>
-        <origin xyz="0 0 0.1" rpy="1.5708 0 0"/>
-    </joint>
-    <link name="base_link">
-        <inertial>
-            <origin xyz="0 0 0" rpy="0 0 0"/>
-            <mass value="1.0"/>
-            <inertia ixx="0.01" ixy="0.0" ixz="0.0" iyy="0.01" iyz="0.0" izz="0.01" />
-        </inertial>
-        <visual>
-            <origin xyz="0 0 0" rpy="0 0 0"/>
-            <geometry>
-                <mesh filename="file://$(find final_assemble_rover_description)/meshes/base_link.stl" />
-            </geometry>
-            <material name="red"/>
-        </visual>
-        <!-- Elevated collision box so the belly doesn't scrape -->
-        <collision>
-            <origin xyz="0 0.05 0" rpy="0 0 0"/>
-            <geometry>
-                <box size="0.1 0.05 0.08"/>
-            </geometry>
-        </collision>
-    </link>
-    <link name="right_wheel_link_1_1">
-        <inertial>
-            <origin xyz="0 0 0" rpy="0 0 0"/>
-            <mass value="0.1"/>
-            <inertia ixx="0.001" ixy="0.0" ixz="0.0" iyy="0.001" iyz="0.0" izz="0.001" />
-        </inertial>
-        <visual>
-            <!-- ORIGINAL OFFSET TO PUSH IT BACK TO THE SIDE -->
-            <origin xyz="0.029 -0.025 -0.06121" rpy="0 0 0"/>
-            <geometry>
-                <mesh filename="file://$(find final_assemble_rover_description)/meshes/right_wheel_link_1.stl" />
-            </geometry>
-            <material name="silver"/>
-        </visual>
-        <collision>
-            <origin xyz="0 0 0" rpy="0 0 0"/>
-            <geometry>
-                <cylinder radius="0.035" length="0.02"/>
-            </geometry>
-        </collision>
-    </link>
-    <joint name="Revolute 19" type="continuous">
-        <origin xyz="-0.029 0.025 0.06121" rpy="0 0 0"/>
-        <parent link="base_link"/>
-        <child link="right_wheel_link_1_1"/>
-        <axis xyz="0.0 0.0 -1.0"/>
-    </joint>
-    <link name="left_wheel_link_1_1">
-        <inertial>
-            <origin xyz="0 0 0" rpy="0 0 0"/>
-            <mass value="0.1"/>
-            <inertia ixx="0.001" ixy="0.0" ixz="0.0" iyy="0.001" iyz="0.0" izz="0.001" />
-        </inertial>
-        <visual>
-            <!-- ORIGINAL OFFSET TO PUSH IT BACK TO THE SIDE -->
-            <origin xyz="0.029 -0.025 0.06121" rpy="0 0 0"/>
-            <geometry>
-                <mesh filename="file://$(find final_assemble_rover_description)/meshes/left_wheel_link_1.stl" />
-            </geometry>
-            <material name="silver"/>
-        </visual>
-        <collision>
-            <origin xyz="0 0 0" rpy="0 0 0"/>
-            <geometry>
-                <cylinder radius="0.035" length="0.02"/>
-            </geometry>
-        </collision>
-    </link>
-    <joint name="Revolute 20" type="continuous">
-        <origin xyz="-0.029 0.025 -0.06121" rpy="0 0 0"/>
-        <parent link="base_link"/>
-        <child link="left_wheel_link_1_1"/>
-        <axis xyz="0.0 0.0 -1.0"/>
-    </joint>
-    <link name="castor_link_1_1">
-        <inertial>
-            <origin xyz="0 0 0" rpy="0 0 0"/>
-            <mass value="0.01"/>
-            <inertia ixx="0.0001" ixy="0.0" ixz="0.0" iyy="0.0001" iyz="0.0" izz="0.0001" />
-        </inertial>
-        <visual>
-            <origin xyz="-0.039746 0.0076 0.0" rpy="0 0 0"/>
-            <geometry>
-                <mesh filename="file://$(find final_assemble_rover_description)/meshes/castor_link_1.stl"/>
-            </geometry>
-            <material name="silver"/>
-        </visual>
-        <collision>
-            <origin xyz="0 0 0" rpy="0 0 0"/>
-            <geometry>
-                <sphere radius="0.002"/>
-            </geometry>
-        </collision>
-    </link>
-    <joint name="Rigid 21" type="fixed">
-        <origin xyz="0.039746 -0.0076 0.0" rpy="0 0 0"/>
-        <parent link="base_link"/>
-        <child link="castor_link_1_1"/>
-    </joint>
-    <link name="laser_link_1_1">
-        <inertial>
-            <origin xyz="0 0 0" rpy="0 0 0"/>
-            <mass value="0.01"/>
-            <inertia ixx="0.0001" ixy="0.0" ixz="0.0" iyy="0.0001" iyz="0.0" izz="0.0001" />
-        </inertial>
-        <visual>
-            <origin xyz="0.0025 -0.09965 -0.0" rpy="0 0 0"/>
-            <geometry>
-                <mesh filename="file://$(find final_assemble_rover_description)/meshes/laser_link_1.stl"/>
-            </geometry>
-            <material name="silver"/>
-        </visual>
-        <collision>
-            <origin xyz="0 0 0" rpy="0 0 0"/>
-            <geometry>
-                <box size="0.03 0.03 0.03"/>
-            </geometry>
-        </collision>
-    </link>
-    <joint name="Rigid 22" type="fixed">
-        <origin xyz="-0.0025 0.09965 0.0" rpy="0 0 0"/>
-        <parent link="base_link"/>
-        <child link="laser_link_1_1"/>
-    </joint>
+<!-- Generated using onshape-to-robot -->
+<!-- Onshape document_id: bf487e698bf759fdcb648406 / workspace_id: 7190dedf85208c03acd2e546 -->
+<robot name="final_assemble_rover">
+  <!-- Link base_link -->
+  <link name="base_link">
+    <inertial>
+      <origin xyz="-0.00490882 -0.000846201 0.0714046" rpy="0 0 0"/>
+      <mass value="0.222325"/>
+      <inertia ixx="0.00059991" ixy="-8.12726e-07" ixz="-3.66324e-05" iyy="0.000620644" iyz="-1.74055e-06" izz="0.00031087"/>
+    </inertial>
+    <!-- Part base_link -->
+    <visual>
+      <origin xyz="0 0 0" rpy="0 -0 0"/>
+      <geometry>
+        <mesh filename="package://assets/base_link.stl"/>
+      </geometry>
+      <material name="base_link_material">
+        <color rgba="0.627451 0.627451 0.627451 1"/>
+      </material>
+    </visual>
+    <collision>
+      <origin xyz="0 0 0" rpy="0 -0 0"/>
+      <geometry>
+        <mesh filename="package://assets/base_link.stl"/>
+      </geometry>
+    </collision>
+    <!-- Part base_link_2 -->
+    <visual>
+      <origin xyz="0 0 0" rpy="0 -0 0"/>
+      <geometry>
+        <mesh filename="package://assets/base_link__2.stl"/>
+      </geometry>
+      <material name="base_link_2_material">
+        <color rgba="0.627451 0.627451 0.627451 1"/>
+      </material>
+    </visual>
+    <collision>
+      <origin xyz="0 0 0" rpy="0 -0 0"/>
+      <geometry>
+        <mesh filename="package://assets/base_link__2.stl"/>
+      </geometry>
+    </collision>
+    <!-- Part base_link_3 -->
+    <visual>
+      <origin xyz="0 0 0" rpy="0 -0 0"/>
+      <geometry>
+        <mesh filename="package://assets/base_link__3.stl"/>
+      </geometry>
+      <material name="base_link_3_material">
+        <color rgba="0.74902 0.74902 0.74902 1"/>
+      </material>
+    </visual>
+    <collision>
+      <origin xyz="0 0 0" rpy="0 -0 0"/>
+      <geometry>
+        <mesh filename="package://assets/base_link__3.stl"/>
+      </geometry>
+    </collision>
+    <!-- Part laser_link_1_1 -->
+    <visual>
+      <origin xyz="0 0 0" rpy="0 -0 0"/>
+      <geometry>
+        <mesh filename="package://assets/laser_link_1_1.stl"/>
+      </geometry>
+      <material name="laser_link_1_1_material">
+        <color rgba="0.627451 0.627451 0.627451 1"/>
+      </material>
+    </visual>
+    <collision>
+      <origin xyz="0 0 0" rpy="0 -0 0"/>
+      <geometry>
+        <mesh filename="package://assets/laser_link_1_1.stl"/>
+      </geometry>
+    </collision>
+    <!-- Part base_link_4 -->
+    <visual>
+      <origin xyz="0 0 0" rpy="0 -0 0"/>
+      <geometry>
+        <mesh filename="package://assets/base_link__4.stl"/>
+      </geometry>
+      <material name="base_link_4_material">
+        <color rgba="0.74902 0.74902 0.74902 1"/>
+      </material>
+    </visual>
+    <collision>
+      <origin xyz="0 0 0" rpy="0 -0 0"/>
+      <geometry>
+        <mesh filename="package://assets/base_link__4.stl"/>
+      </geometry>
+    </collision>
+    <!-- Part base_link_5 -->
+    <visual>
+      <origin xyz="0 0 0" rpy="0 -0 0"/>
+      <geometry>
+        <mesh filename="package://assets/base_link__5.stl"/>
+      </geometry>
+      <material name="base_link_5_material">
+        <color rgba="1 0.807843 0.498039 1"/>
+      </material>
+    </visual>
+    <collision>
+      <origin xyz="0 0 0" rpy="0 -0 0"/>
+      <geometry>
+        <mesh filename="package://assets/base_link__5.stl"/>
+      </geometry>
+    </collision>
+    <!-- Part base_link_6 -->
+    <visual>
+      <origin xyz="0 0 0" rpy="0 -0 0"/>
+      <geometry>
+        <mesh filename="package://assets/base_link__6.stl"/>
+      </geometry>
+      <material name="base_link_6_material">
+        <color rgba="0.627451 0.627451 0.627451 1"/>
+      </material>
+    </visual>
+    <collision>
+      <origin xyz="0 0 0" rpy="0 -0 0"/>
+      <geometry>
+        <mesh filename="package://assets/base_link__6.stl"/>
+      </geometry>
+    </collision>
+    <!-- Part base_link_7 -->
+    <visual>
+      <origin xyz="0 0 0" rpy="0 -0 0"/>
+      <geometry>
+        <mesh filename="package://assets/base_link__7.stl"/>
+      </geometry>
+      <material name="base_link_7_material">
+        <color rgba="0.627451 0.627451 0.627451 1"/>
+      </material>
+    </visual>
+    <collision>
+      <origin xyz="0 0 0" rpy="0 -0 0"/>
+      <geometry>
+        <mesh filename="package://assets/base_link__7.stl"/>
+      </geometry>
+    </collision>
+    <!-- Part base_link_8 -->
+    <visual>
+      <origin xyz="0 0 0" rpy="0 -0 0"/>
+      <geometry>
+        <mesh filename="package://assets/base_link__8.stl"/>
+      </geometry>
+      <material name="base_link_8_material">
+        <color rgba="1 0.956863 0.886275 1"/>
+      </material>
+    </visual>
+    <collision>
+      <origin xyz="0 0 0" rpy="0 -0 0"/>
+      <geometry>
+        <mesh filename="package://assets/base_link__8.stl"/>
+      </geometry>
+    </collision>
+    <!-- Part base_link_9 -->
+    <visual>
+      <origin xyz="0 0 0" rpy="0 -0 0"/>
+      <geometry>
+        <mesh filename="package://assets/base_link__9.stl"/>
+      </geometry>
+      <material name="base_link_9_material">
+        <color rgba="0.627451 0.627451 0.627451 1"/>
+      </material>
+    </visual>
+    <collision>
+      <origin xyz="0 0 0" rpy="0 -0 0"/>
+      <geometry>
+        <mesh filename="package://assets/base_link__9.stl"/>
+      </geometry>
+    </collision>
+    <!-- Part base_link_10 -->
+    <visual>
+      <origin xyz="0 0 0" rpy="0 -0 0"/>
+      <geometry>
+        <mesh filename="package://assets/base_link__10.stl"/>
+      </geometry>
+      <material name="base_link_10_material">
+        <color rgba="0.627451 0.627451 0.627451 1"/>
+      </material>
+    </visual>
+    <collision>
+      <origin xyz="0 0 0" rpy="0 -0 0"/>
+      <geometry>
+        <mesh filename="package://assets/base_link__10.stl"/>
+      </geometry>
+    </collision>
+    <!-- Part base_link_11 -->
+    <visual>
+      <origin xyz="0 0 0" rpy="0 -0 0"/>
+      <geometry>
+        <mesh filename="package://assets/base_link__11.stl"/>
+      </geometry>
+      <material name="base_link_11_material">
+        <color rgba="0.627451 0.627451 0.627451 1"/>
+      </material>
+    </visual>
+    <collision>
+      <origin xyz="0 0 0" rpy="0 -0 0"/>
+      <geometry>
+        <mesh filename="package://assets/base_link__11.stl"/>
+      </geometry>
+    </collision>
+    <!-- Part base_link_12 -->
+    <visual>
+      <origin xyz="0 0 0" rpy="0 -0 0"/>
+      <geometry>
+        <mesh filename="package://assets/base_link__12.stl"/>
+      </geometry>
+      <material name="base_link_12_material">
+        <color rgba="1 0.807843 0.498039 1"/>
+      </material>
+    </visual>
+    <collision>
+      <origin xyz="0 0 0" rpy="0 -0 0"/>
+      <geometry>
+        <mesh filename="package://assets/base_link__12.stl"/>
+      </geometry>
+    </collision>
+    <!-- Part base_link_13 -->
+    <visual>
+      <origin xyz="0 0 0" rpy="0 -0 0"/>
+      <geometry>
+        <mesh filename="package://assets/base_link__13.stl"/>
+      </geometry>
+      <material name="base_link_13_material">
+        <color rgba="0.627451 0.627451 0.627451 1"/>
+      </material>
+    </visual>
+    <collision>
+      <origin xyz="0 0 0" rpy="0 -0 0"/>
+      <geometry>
+        <mesh filename="package://assets/base_link__13.stl"/>
+      </geometry>
+    </collision>
+    <!-- Part base_link_14 -->
+    <visual>
+      <origin xyz="0 0 0" rpy="0 -0 0"/>
+      <geometry>
+        <mesh filename="package://assets/base_link__14.stl"/>
+      </geometry>
+      <material name="base_link_14_material">
+        <color rgba="0.627451 0.627451 0.627451 1"/>
+      </material>
+    </visual>
+    <collision>
+      <origin xyz="0 0 0" rpy="0 -0 0"/>
+      <geometry>
+        <mesh filename="package://assets/base_link__14.stl"/>
+      </geometry>
+    </collision>
+    <!-- Part base_link_15 -->
+    <visual>
+      <origin xyz="0 0 0" rpy="0 -0 0"/>
+      <geometry>
+        <mesh filename="package://assets/base_link__15.stl"/>
+      </geometry>
+      <material name="base_link_15_material">
+        <color rgba="0.627451 0.627451 0.627451 1"/>
+      </material>
+    </visual>
+    <collision>
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
Commit message: xacro update

File: final_assemble_rover_description/urdf/final_assemble_rover.xacro (robot description, xacro)
@@ -1,6 +1,16 @@
 <?xml version="1.0" ?>
-<!-- Generated using onshape-to-robot -->
-<!-- Onshape document_id: bf487e698bf759fdcb648406 / workspace_id: 7190dedf85208c03acd2e546 -->
-<robot name="final_assemble_rover">
+<robot name="final_assemble_rover" xmlns:xacro="http://www.ros.org/wiki/xacro">
+    <!-- GAZEBO PLUGINS & MATERIALS -->
+    <xacro:include filename="$(find final_assemble_rover_description)/urdf/materials.xacro" />
+    <xacro:include filename="$(find final_assemble_rover_description)/urdf/final_assemble_rover.trans" />
+    <xacro:include filename="$(find final_assemble_rover_description)/urdf/final_assemble_rover.gazebo" />
+    <xacro:include filename="$(find final_assemble_rover_description)/urdf/gazebo_control.xacro" />
+    <!-- NAV STACK ROOT LINK -->
+    <link name="base_footprint"/>
+    <joint name="base_footprint_joint" type="fixed">
+        <parent link="base_footprint"/>
+        <child link="base_link"/>
+        <origin xyz="0 0 0.1" rpy="0 0 0"/>
+    </joint>
   <!-- Link base_link -->
   <link name="base_link">
