Commit message: xacro_overwrite

File: final_assemble_rover_description/urdf/final_assemble_rover.xacro (robot description, xacro)
@@ -24,5 +24,5 @@
       <origin xyz="0 0 0" rpy="0 -0 0"/>
       <geometry>
-        <mesh filename="package://assets/base_link.stl"/>
+        <mesh filename="final_assemble_rover_description/meshesbase_link.stl"/>
       </geometry>
       <material name="base_link_material">
@@ -33,5 +33,5 @@
       <origin xyz="0 0 0" rpy="0 -0 0"/>
       <geometry>
-        <mesh filename="package://assets/base_link.stl"/>
+        <mesh filename="final_assemble_rover_description/meshesbase_link.stl"/>
       </geometry>
     </collision>
@@ -40,5 +40,5 @@
       <origin xyz="0 0 0" rpy="0 -0 0"/>
       <geometry>
-        <mesh filename="package://assets/base_link__2.stl"/>
+        <mesh filename="final_assemble_rover_description/meshesbase_link__2.stl"/>
       </geometry>
       <material name="base_link_2_material">
@@ -49,5 +49,5 @@
       <origin xyz="0 0 0" rpy="0 -0 0"/>
       <geometry>
-        <mesh filename="package://assets/base_link__2.stl"/>
+        <mesh filename="final_assemble_rover_description/meshesbase_link__2.stl"/>
       </geometry>
     </collision>
@@ -56,5 +56,5 @@
       <origin xyz="0 0 0" rpy="0 -0 0"/>
       <geometry>
-        <mesh filename="package://assets/base_link__3.stl"/>
+        <mesh filename="final_assemble_rover_description/meshesbase_link__3.stl"/>
       </geometry>
       <material name="base_link_3_material">
@@ -65,5 +65,5 @@
       <origin xyz="0 0 0" rpy="0 -0 0"/>
       <geometry>
-        <mesh filename="package://assets/base_link__3.stl"/>
+        <mesh filename="final_assemble_rover_description/meshesbase_link__3.stl"/>
       </geometry>
     </collision>
@@ -72,5 +72,5 @@
       <origin xyz="0 0 0" rpy="0 -0 0"/>
       <geometry>
-        <mesh filename="package://assets/laser_link_1_1.stl"/>
+        <mesh filename="final_assemble_rover_description/mesheslaser_link_1_1.stl"/>
       </geometry>
       <material name="laser_link_1_1_material">
@@ -81,5 +81,5 @@
       <origin xyz="0 0 0" rpy="0 -0 0"/>
       <geometry>
-        <mesh filename="package://assets/laser_link_1_1.stl"/>
+        <mesh filename="final_assemble_rover_description/mesheslaser_link_1_1.stl"/>
       </geometry>
     </collision>
@@ -88,5 +88,5 @@
       <origin xyz="0 0 0" rpy="0 -0 0"/>
       <geometry>
-        <mesh filename="package://assets/base_link__4.stl"/>
+        <mesh filename="final_assemble_rover_description/meshesbase_link__4.stl"/>
       </geometry>
       <material name="base_link_4_material">
@@ -97,5 +97,5 @@
       <origin xyz="0 0 0" rpy="0 -0 0"/>
       <geometry>
-        <mesh filename="package://assets/base_link__4.stl"/>
+        <mesh filename="final_assemble_rover_description/meshesbase_link__4.stl"/>
       </geometry>
     </collision>
@@ -104,5 +104,5 @@
       <origin xyz="0 0 0" rpy="0 -0 0"/>
       <geometry>
-        <mesh filename="package://assets/base_link__5.stl"/>
+        <mesh filename="final_assemble_rover_description/meshesbase_link__5.stl"/>
       </geometry>
       <material name="base_link_5_material">
@@ -113,5 +113,5 @@
       <origin xyz="0 0 0" rpy="0 -0 0"/>
       <geometry>
-        <mesh filename="package://assets/base_link__5.stl"/>
+        <mesh filename="final_assemble_rover_description/meshesbase_link__5.stl"/>
       </geometry>
     </collision>
@@ -120,5 +120,5 @@
       <origin xyz="0 0 0" rpy="0 -0 0"/>
       <geometry>
-        <mesh filename="package://assets/base_link__6.stl"/>
+        <mesh filename="final_assemble_rover_description/meshesbase_link__6.stl"/>
       </geometry>
       <material name="base_link_6_material">
@@ -129,5 +129,5 @@
       <origin xyz="0 0 0" rpy="0 -0 0"/>
       <geometry>
-        <mesh filename="package://assets/base_link__6.stl"/>
+        <mesh filename="final_assemble_rover_description/meshesbase_link__6.stl"/>
       </geometry>
     </collision>
@@ -136,5 +136,5 @@
       <origin xyz="0 0 0" rpy="0 -0 0"/>
       <geometry>
-        <mesh filename="package://assets/base_link__7.stl"/>
+        <mesh filename="final_assemble_rover_description/meshesbase_link__7.stl"/>
       </geometry>
       <material name="base_link_7_material">
@@ -145,5 +145,5 @@
       <origin xyz="0 0 0" rpy="0 -0 0"/>
       <geometry>
-        <mesh filename="package://assets/base_link__7.stl"/>
+        <mesh filename="final_assemble_rover_description/meshesbase_link__7.stl"/>
       </geometry>
     </collision>
@@ -152,5 +152,5 @@
       <origin xyz="0 0 0" rpy="0 -0 0"/>
       <geometry>
-        <mesh filename="package://assets/base_link__8.stl"/>
+        <mesh filename="final_assemble_rover_description/meshesbase_link__8.stl"/>
       </geometry>
       <material name="base_link_8_material">
@@ -161,5 +161,5 @@
       <origin xyz="0 0 0" rpy="0 -0 0"/>
       <geometry>
-        <mesh filename="package://assets/base_link__8.stl"/>
+        <mesh filename="final_assemble_rover_description/meshesbase_link__8.stl"/>
       </geometry>
     </collision>
@@ -168,5 +168,5 @@
       <origin xyz="0 0 0" rpy="0 -0 0"/>
       <geometry>
-        <mesh filename="package://assets/base_link__9.stl"/>
+        <mesh filename="final_assemble_rover_description/meshesbase_link__9.stl"/>
       </geometry>
       <material name="base_link_9_material">
@@ -177,5 +177,5 @@
       <origin xyz="0 0 0" rpy="0 -0 0"/>
       <geometry>
-        <mesh filename="package://assets/base_link__9.stl"/>
+        <mesh filename="final_assemble_rover_description/meshesbase_link__9.stl"/>
       </geometry>
     </collision>
@@ -184,5 +184,5 @@
       <origin xyz="0 0 0" rpy="0 -0 0"/>
       <geometry>
-        <mesh filename="package://assets/base_link__10.stl"/>
+        <mesh filename="final_assemble_rover_description/meshesbase_link__10.stl"/>
       </geometry>
       <material name="base_link_10_material">
@@ -193,5 +193,5 @@
       <origin xyz="0 0 0" rpy="0 -0 0"/>
       <geometry>
-        <mesh filename="package://assets/base_link__10.stl"/>
+        <mesh filename="final_assemble_rover_description/meshesbase_link__10.stl"/>
       </geometry>
     </collision>
@@ -200,5 +200,5 @@
       <origin xyz="0 0 0" rpy="0 -0 0"/>
       <geometry>
-        <mesh filename="package://assets/base_link__11.stl"/>
+        <mesh filename="final_assemble_rover_description/meshesbase_link__11.stl"/>
       </geometry>
       <material name="base_link_11_material">
@@ -209,5 +209,5 @@
       <origin xyz="0 0 0" rpy="0 -0 0"/>
       <geometry>
-        <mesh filename="package://assets/base_link__11.stl"/>
+        <mesh filename="final_assemble_rover_description/meshesbase_link__11.stl"/>
       </geometry>
     </collision>
@@ -216,5 +216,5 @@
       <origin xyz="0 0 0" rpy="0 -0 0"/>
       <geometry>
-        <mesh filename="package://assets/base_link__12.stl"/>
+        <mesh filename="final_assemble_rover_description/meshesbase_link__12.stl"/>
       </geometry>
       <material name="base_link_12_material">
@@ -225,5 +225,5 @@
       <origin xyz="0 0 0" rpy="0 -0 0"/>
       <geometry>
-        <mesh filename="package://assets/base_link__12.stl"/>
+        <mesh filename="final_assemble_rover_description/meshesbase_link__12.stl"/>
       </geometry>
     </collision>
@@ -232,5 +232,5 @@
       <origin xyz="0 0 0" rpy="0 -0 0"/>
       <geometry>
-        <mesh filename="package://assets/base_link__13.stl"/>
+        <mesh filename="final_assemble_rover_description/meshesbase_link__13.stl"/>
       </geometry>
       <material name="base_link_13_material">
@@ -241,5 +241,5 @@
       <origin xyz="0 0 0" rpy="0 -0 0"/>
       <geometry>
-        <mesh filename="package://assets/base_link__13.stl"/>
+        <mesh filename="final_assemble_rover_description/meshesbase_link__13.stl"/>
       </geometry>
     </collision>
@@ -248,5 +248,5 @@
       <origin xyz="0 0 0" rpy="0 -0 0"/>
       <geometry>
-        <mesh filename="package://assets/base_link__14.stl"/>
+        <mesh filename="final_assemble_rover_description/meshesbase_link__14.stl"/>
       </geometry>
       <material name="base_link_14_material">
@@ -257,5 +257,5 @@
       <origin xyz="0 0 0" rpy="0 -0 0"/>
       <geometry>
-        <mesh filename="package://assets/base_link__14.stl"/>
+        <mesh filename="final_assemble_rover_description/meshesbase_link__14.stl"/>
       </geometry>
     </collision>
@@ -264,5 +264,5 @@
       <origin xyz="0 0 0" rpy="0 -0 0"/>
       <geometry>
-        <mesh filename="package://assets/base_link__15.stl"/>
+        <mesh filename="final_assemble_rover_description/meshesbase_link__15.stl"/>
       </geometry>
       <material name="base_link_15_material">
@@ -273,5 +273,5 @@
       <origin xyz="0 0 0" rpy="0 -0 0"/>
       <geometry>
-        <mesh filename="package://assets/base_link__15.stl"/>
+        <mesh filename="final_assemble_rover_description/meshesbase_link__15.stl"/>
       </geometry>
     </collision>
@@ -280,5 +280,5 @@
       <origin xyz="0 0 0" rpy="0 -0 0"/>
       <geometry>
-        <mesh filename="package://assets/laser_link_1_1__2.stl"/>
+        <mesh filename="final_assemble_rover_description/mesheslaser_link_1_1__2.stl"/>
       </geometry>
       <material name="laser_link_1_1_2_material">
@@ -289,5 +289,5 @@
       <origin xyz="0 0 0" rpy="0 -0 0"/>
       <geometry>
-        <mesh filename="package://assets/laser_link_1_1__2.stl"/>
+        <mesh filename="final_assemble_rover_description/mesheslaser_link_1_1__2.stl"/>
       </geometry>
     </collision>
@@ -296,5 +296,5 @@
       <origin xyz="0 0 0" rpy="0 -0 0"/>
       <geometry>
-        <mesh filename="package://assets/base_link__16.stl"/>
+        <mesh filename="final_assemble_rover_description/meshesbase_link__16.stl"/>
       </geometry>
       <material name="base_link_16_material">
@@ -305,5 +305,5 @@
       <origin xyz="0 0 0" rpy="0 -0 0"/>
       <geometry>
-        <mesh filename="package://assets/base_link__16.stl"/>
+        <mesh filename="final_assemble_rover_description/meshesbase_link__16.stl"/>
       </geometry>
     </collision>
@@ -312,5 +312,5 @@
       <origin xyz="0 0 0" rpy="0 -0 0"/>
       <geometry>
-        <mesh filename="package://assets/base_link__17.stl"/>
+        <mesh filename="final_assemble_rover_description/meshesbase_link__17.stl"/>
       </geometry>
       <material name="base_link_17_material">
@@ -321,5 +321,5 @@
       <origin xyz="0 0 0" rpy="0 -0 0"/>
       <geometry>
-        <mesh filename="package://assets/base_link__17.stl"/>
+        <mesh filename="final_assemble_rover_description/meshesbase_link__17.stl"/>
       </geometry>
     </collision>
@@ -328,5 +328,5 @@
       <origin xyz="0 0 0" rpy="0 -0 0"/>
       <geometry>
-        <mesh filename="package://assets/base_link__18.stl"/>
+        <mesh filename="final_assemble_rover_description/meshesbase_link__18.stl"/>
       </geometry>
       <material name="base_link_18_material">
@@ -337,5 +337,5 @@
       <origin xyz="0 0 0" rpy="0 -0 0"/>
       <geometry>
-        <mesh filename="package://assets/base_link__18.stl"/>
+        <mesh filename="final_assemble_rover_description/meshesbase_link__18.stl"/>
       </geometry>
     </collision>
@@ -344,5 +344,5 @@
       <origin xyz="0 0 0" rpy="0 -0 0"/>
       <geometry>
-        <mesh filename="package://assets/base_link__19.stl"/>
+        <mesh filename="final_assemble_rover_description/meshesbase_link__19.stl"/>
       </geometry>
       <material name="base_link_19_material">
@@ -353,5 +353,5 @@
       <origin xyz="0 0 0" rpy="0 -0 0"/>
       <geometry>
-        <mesh filename="package://assets/base_link__19.stl"/>
+        <mesh filename="final_assemble_rover_description/meshesbase_link__19.stl"/>
       </geometry>
     </collision>
@@ -360,5 +360,5 @@
       <origin xyz="0 0 0" rpy="0 -0 0"/>
       <geometry>
-        <mesh filename="package://assets/base_link__20.stl"/>
+        <mesh filename="final_assemble_rover_description/meshesbase_link__20.stl"/>
       </geometry>
       <material name="base_link_20_material">
@@ -369,5 +369,5 @@
       <origin xyz="0 0 0" rpy="0 -0 0"/>
       <geometry>
-        <mesh filename="package://assets/base_link__20.stl"/>
+        <mesh filename="final_assemble_rover_description/meshesbase_link__20.stl"/>
       </geometry>
     </collision>
@@ -376,5 +376,5 @@
       <origin xyz="0 0 0" rpy="0 -0 0"/>
       <geometry>
-        <mesh filename="package://assets/base_link__21.stl"/>
+        <mesh filename="final_assemble_rover_description/meshesbase_link__21.stl"/>
       </geometry>
       <material name="base_link_21_material">
@@ -385,5 +385,5 @@
       <origin xyz="0 0 0" rpy="0 -0 0"/>
       <geometry>
-        <mesh filename="package://assets/base_link__21.stl"/>
+        <mesh filename="final_assemble_rover_description/meshesbase_link__21.stl"/>
       </geometry>
     </collision>
@@ -392,5 +392,5 @@
       <origin xyz="0 0 0" rpy="0 -0 0"/>
       <geometry>
-        <mesh filename="package://assets/base_link__22.stl"/>
+        <mesh filename="final_assemble_rover_description/meshesbase_link__22.stl"/>
       </geometry>
       <material name="base_link_22_material">
@@ -401,5 +401,5 @@
       <origin xyz="0 0 0" rpy="0 -0 0"/>
       <geometry>
-        <mesh filename="package://assets/base_link__22.stl"/>
+        <mesh filename="final_assemble_rover_description/meshesbase_link__22.stl"/>
       </geometry>
     </collision>
@@ -408,5 +408,5 @@
       <origin xyz="0 0 0" rpy="0 -0 0"/>
       <geometry>
-        <mesh filename="package://assets/base_link__23.stl"/>
+        <mesh filename="final_assemble_rover_description/meshesbase_link__23.stl"/>
       </geometry>
       <material name="base_link_23_material">
@@ -417,5 +417,5 @@
       <origin xyz="0 0 0" rpy="0 -0 0"/>
       <geometry>
-        <mesh filename="package://assets/base_link__23.stl"/>
+        <mesh filename="final_assemble_rover_description/meshesbase_link__23.stl"/>
       </geometry>
     </collision>
@@ -424,5 +424,5 @@
       <origin xyz="0 0 0" rpy="0 -0 0"/>
       <geometry>
-        <mesh filename="package://assets/base_link__24.stl"/>
+        <mesh filename="final_assemble_rover_description/meshesbase_link__24.stl"/>
       </geometry>
       <material name="base_link_24_material">
@@ -433,5 +433,5 @@
       <origin xyz="0 0 0" rpy="0 -0 0"/>
       <geometry>
-        <mesh filename="package://assets/base_link__24.stl"/>
+        <mesh filename="final_assemble_rover_description/meshesbase_link__24.stl"/>
       </geometry>
     </collision>
@@ -440,5 +440,5 @@
       <origin xyz="0 0 0" rpy="0 -0 0"/>
       <geometry>
-        <mesh filename="package://assets/laser_link_1_1__3.stl"/>
+        <mesh filename="final_assemble_rover_description/mesheslaser_link_1_1__3.stl"/>
       </geometry>
       <material name="laser_link_1_1_3_material">
@@ -449,5 +449,5 @@
       <origin xyz="0 0 0" rpy="0 -0 0"/>
       <geometry>
-        <mesh filename="package://assets/laser_link_1_1__3.stl"/>
+        <mesh filename="final_assemble_rover_description/mesheslaser_link_1_1__3.stl"/>
       </geometry>
     </collision>
@@ -456,5 +456,5 @@
       <origin xyz="0 0 0" rpy="0 -0 0"/>
       <geometry>
-        <mesh filename="package://assets/base_link__25.stl"/>
+        <mesh filename="final_assemble_rover_description/meshesbase_link__25.stl"/>
       </geometry>
       <material name="base_link_25_material">
@@ -465,5 +465,5 @@
       <origin xyz="0 0 0" rpy="0 -0 0"/>
       <geometry>
-        <mesh filename="package://assets/base_link__25.stl"/>
+        <mesh filename="final_assemble_rover_description/meshesbase_link__25.stl"/>
       </geometry>
     </collision>
@@ -472,5 +472,5 @@
       <origin xyz="0 0 0" rpy="0 -0 0"/>
       <geometry>
-        <mesh filename="package://assets/base_link__26.stl"/>
+        <mesh filename="final_assemble_rover_description/meshesbase_link__26.stl"/>
       </geometry>
       <material name="base_link_26_material">
@@ -481,5 +481,5 @@
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