Commit message: retrace

File: final_assemble_rover_description/urdf/final_assemble_rover.xacro (robot description, xacro)
@@ -1,16 +1,6 @@
 <?xml version="1.0" ?>
-<robot name="final_assemble_rover" xmlns:xacro="http://www.ros.org/wiki/xacro">
-    <!-- GAZEBO PLUGINS & MATERIALS -->
-    <xacro:include filename="$(find final_assemble_rover_description)/urdf/materials.xacro" />
-    <xacro:include filename="$(find final_assemble_rover_description)/urdf/final_assemble_rover.trans" />
-    <xacro:include filename="$(find final_assemble_rover_description)/urdf/final_assemble_rover.gazebo" />
-    <xacro:include filename="$(find final_assemble_rover_description)/urdf/gazebo_control.xacro" />
-    <!-- NAV STACK ROOT LINK -->
-    <link name="base_footprint"/>
-    <joint name="base_footprint_joint" type="fixed">
-        <parent link="base_footprint"/>
-        <child link="base_link"/>
-        <origin xyz="0 0 0.1" rpy="0 0 0"/>
-    </joint>
+<!-- Generated using onshape-to-robot -->
+<!-- Onshape document_id: bf487e698bf759fdcb648406 / workspace_id: 7190dedf85208c03acd2e546 -->
+<robot name="onshape_rover_files">
   <!-- Link base_link -->
   <link name="base_link">
@@ -24,5 +14,5 @@
       <origin xyz="0 0 0" rpy="0 -0 0"/>
       <geometry>
-        <mesh filename="final_assemble_rover_description/meshesbase_link.stl"/>
+        <mesh filename="package://assets/base_link.stl"/>
       </geometry>
       <material name="base_link_material">
@@ -33,5 +23,5 @@
       <origin xyz="0 0 0" rpy="0 -0 0"/>
       <geometry>
-        <mesh filename="final_assemble_rover_description/meshesbase_link.stl"/>
+        <mesh filename="package://assets/base_link.stl"/>
       </geometry>
     </collision>
@@ -40,5 +30,5 @@
       <origin xyz="0 0 0" rpy="0 -0 0"/>
       <geometry>
-        <mesh filename="final_assemble_rover_description/meshesbase_link__2.stl"/>
+        <mesh filename="package://assets/base_link__2.stl"/>
       </geometry>
       <material name="base_link_2_material">
@@ -49,5 +39,5 @@
       <origin xyz="0 0 0" rpy="0 -0 0"/>
       <geometry>
-        <mesh filename="final_assemble_rover_description/meshesbase_link__2.stl"/>
+        <mesh filename="package://assets/base_link__2.stl"/>
       </geometry>
     </collision>
@@ -56,5 +46,5 @@
       <origin xyz="0 0 0" rpy="0 -0 0"/>
       <geometry>
-        <mesh filename="final_assemble_rover_description/meshesbase_link__3.stl"/>
+        <mesh filename="package://assets/base_link__3.stl"/>
       </geometry>
       <material name="base_link_3_material">
@@ -65,5 +55,5 @@
       <origin xyz="0 0 0" rpy="0 -0 0"/>
       <geometry>
-        <mesh filename="final_assemble_rover_description/meshesbase_link__3.stl"/>
+        <mesh filename="package://assets/base_link__3.stl"/>
       </geometry>
     </collision>
@@ -72,5 +62,5 @@
       <origin xyz="0 0 0" rpy="0 -0 0"/>
       <geometry>
-        <mesh filename="final_assemble_rover_description/mesheslaser_link_1_1.stl"/>
+        <mesh filename="package://assets/laser_link_1_1.stl"/>
       </geometry>
       <material name="laser_link_1_1_material">
@@ -81,5 +71,5 @@
       <origin xyz="0 0 0" rpy="0 -0 0"/>
       <geometry>
-        <mesh filename="final_assemble_rover_description/mesheslaser_link_1_1.stl"/>
+        <mesh filename="package://assets/laser_link_1_1.stl"/>
       </geometry>
     </collision>
@@ -88,5 +78,5 @@
       <origin xyz="0 0 0" rpy="0 -0 0"/>
       <geometry>
-        <mesh filename="final_assemble_rover_description/meshesbase_link__4.stl"/>
+        <mesh filename="package://assets/base_link__4.stl"/>
       </geometry>
       <material name="base_link_4_material">
@@ -97,5 +87,5 @@
       <origin xyz="0 0 0" rpy="0 -0 0"/>
       <geometry>
-        <mesh filename="final_assemble_rover_description/meshesbase_link__4.stl"/>
+        <mesh filename="package://assets/base_link__4.stl"/>
       </geometry>
     </collision>
@@ -104,5 +94,5 @@
       <origin xyz="0 0 0" rpy="0 -0 0"/>
       <geometry>
-        <mesh filename="final_assemble_rover_description/meshesbase_link__5.stl"/>
+        <mesh filename="package://assets/base_link__5.stl"/>
       </geometry>
       <material name="base_link_5_material">
@@ -113,5 +103,5 @@
       <origin xyz="0 0 0" rpy="0 -0 0"/>
       <geometry>
-        <mesh filename="final_assemble_rover_description/meshesbase_link__5.stl"/>
+        <mesh filename="package://assets/base_link__5.stl"/>
       </geometry>
     </collision>
@@ -120,5 +110,5 @@
       <origin xyz="0 0 0" rpy="0 -0 0"/>
       <geometry>
-        <mesh filename="final_assemble_rover_description/meshesbase_link__6.stl"/>
+        <mesh filename="package://assets/base_link__6.stl"/>
       </geometry>
       <material name="base_link_6_material">
@@ -129,5 +119,5 @@
       <origin xyz="0 0 0" rpy="0 -0 0"/>
       <geometry>
-        <mesh filename="final_assemble_rover_description/meshesbase_link__6.stl"/>
+        <mesh filename="package://assets/base_link__6.stl"/>
       </geometry>
     </collision>
@@ -136,5 +126,5 @@
       <origin xyz="0 0 0" rpy="0 -0 0"/>
       <geometry>
-        <mesh filename="final_assemble_rover_description/meshesbase_link__7.stl"/>
+        <mesh filename="package://assets/base_link__7.stl"/>
       </geometry>
       <material name="base_link_7_material">
@@ -145,5 +135,5 @@
       <origin xyz="0 0 0" rpy="0 -0 0"/>
       <geometry>
-        <mesh filename="final_assemble_rover_description/meshesbase_link__7.stl"/>
+        <mesh filename="package://assets/base_link__7.stl"/>
       </geometry>
     </collision>
@@ -152,5 +142,5 @@
       <origin xyz="0 0 0" rpy="0 -0 0"/>
       <geometry>
-        <mesh filename="final_assemble_rover_description/meshesbase_link__8.stl"/>
+        <mesh filename="package://assets/base_link__8.stl"/>
       </geometry>
       <material name="base_link_8_material">
@@ -161,5 +151,5 @@
       <origin xyz="0 0 0" rpy="0 -0 0"/>
       <geometry>
-        <mesh filename="final_assemble_rover_description/meshesbase_link__8.stl"/>
+        <mesh filename="package://assets/base_link__8.stl"/>
       </geometry>
     </collision>
@@ -168,5 +158,5 @@
       <origin xyz="0 0 0" rpy="0 -0 0"/>
       <geometry>
-        <mesh filename="final_assemble_rover_description/meshesbase_link__9.stl"/>
+        <mesh filename="package://assets/base_link__9.stl"/>
       </geometry>
       <material name="base_link_9_material">
@@ -177,5 +167,5 @@
       <origin xyz="0 0 0" rpy="0 -0 0"/>
       <geometry>
-        <mesh filename="final_assemble_rover_description/meshesbase_link__9.stl"/>
+        <mesh filename="package://assets/base_link__9.stl"/>
       </geometry>
     </collision>
@@ -184,5 +174,5 @@
       <origin xyz="0 0 0" rpy="0 -0 0"/>
       <geometry>
-        <mesh filename="final_assemble_rover_description/meshesbase_link__10.stl"/>
+        <mesh filename="package://assets/base_link__10.stl"/>
       </geometry>
       <material name="base_link_10_material">
@@ -193,5 +183,5 @@
       <origin xyz="0 0 0" rpy="0 -0 0"/>
       <geometry>
-        <mesh filename="final_assemble_rover_description/meshesbase_link__10.stl"/>
+        <mesh filename="package://assets/base_link__10.stl"/>
       </geometry>
     </collision>
@@ -200,5 +190,5 @@
       <origin xyz="0 0 0" rpy="0 -0 0"/>
       <geometry>
-        <mesh filename="final_assemble_rover_description/meshesbase_link__11.stl"/>
+        <mesh filename="package://assets/base_link__11.stl"/>
       </geometry>
       <material name="base_link_11_material">
@@ -209,5 +199,5 @@
       <origin xyz="0 0 0" rpy="0 -0 0"/>
       <geometry>
-        <mesh filename="final_assemble_rover_description/meshesbase_link__11.stl"/>
+        <mesh filename="package://assets/base_link__11.stl"/>
       </geometry>
     </collision>
@@ -216,5 +206,5 @@
       <origin xyz="0 0 0" rpy="0 -0 0"/>
       <geometry>
-        <mesh filename="final_assemble_rover_description/meshesbase_link__12.stl"/>
+        <mesh filename="package://assets/base_link__12.stl"/>
       </geometry>
       <material name="base_link_12_material">
@@ -225,5 +215,5 @@
       <origin xyz="0 0 0" rpy="0 -0 0"/>
       <geometry>
-        <mesh filename="final_assemble_rover_description/meshesbase_link__12.stl"/>
+        <mesh filename="package://assets/base_link__12.stl"/>
       </geometry>
     </collision>
@@ -232,5 +222,5 @@
       <origin xyz="0 0 0" rpy="0 -0 0"/>
       <geometry>
-        <mesh filename="final_assemble_rover_description/meshesbase_link__13.stl"/>
+        <mesh filename="package://assets/base_link__13.stl"/>
       </geometry>
       <material name="base_link_13_material">
@@ -241,5 +231,5 @@
       <origin xyz="0 0 0" rpy="0 -0 0"/>
       <geometry>
-        <mesh filename="final_assemble_rover_description/meshesbase_link__13.stl"/>
+        <mesh filename="package://assets/base_link__13.stl"/>
       </geometry>
     </collision>
@@ -248,5 +238,5 @@
       <origin xyz="0 0 0" rpy="0 -0 0"/>
       <geometry>
-        <mesh filename="final_assemble_rover_description/meshesbase_link__14.stl"/>
+        <mesh filename="package://assets/base_link__14.stl"/>
       </geometry>
       <material name="base_link_14_material">
@@ -257,5 +247,5 @@
       <origin xyz="0 0 0" rpy="0 -0 0"/>
       <geometry>
-        <mesh filename="final_assemble_rover_description/meshesbase_link__14.stl"/>
+        <mesh filename="package://assets/base_link__14.stl"/>
       </geometry>
     </collision>
@@ -264,5 +254,5 @@
       <origin xyz="0 0 0" rpy="0 -0 0"/>
       <geometry>
-        <mesh filename="final_assemble_rover_description/meshesbase_link__15.stl"/>
+        <mesh filename="package://assets/base_link__15.stl"/>
       </geometry>
       <material name="base_link_15_material">
@@ -273,5 +263,5 @@
       <origin xyz="0 0 0" rpy="0 -0 0"/>
       <geometry>
-        <mesh filename="final_assemble_rover_description/meshesbase_link__15.stl"/>
+        <mesh filename="package://assets/base_link__15.stl"/>
       </geometry>
     </collision>
@@ -280,5 +270,5 @@
       <origin xyz="0 0 0" rpy="0 -0 0"/>
       <geometry>
-        <mesh filename="final_assemble_rover_description/mesheslaser_link_1_1__2.stl"/>
+        <mesh filename="package://assets/laser_link_1_1__2.stl"/>
       </geometry>
       <material name="laser_link_1_1_2_material">
@@ -289,5 +279,5 @@
       <origin xyz="0 0 0" rpy="0 -0 0"/>
       <geometry>
-        <mesh filename="final_assemble_rover_description/mesheslaser_link_1_1__2.stl"/>
+        <mesh filename="package://assets/laser_link_1_1__2.stl"/>
       </geometry>
     </collision>
@@ -296,5 +286,5 @@
       <origin xyz="0 0 0" rpy="0 -0 0"/>
       <geometry>
-        <mesh filename="final_assemble_rover_description/meshesbase_link__16.stl"/>
+        <mesh filename="package://assets/base_link__16.stl"/>
       </geometry>
       <material name="base_link_16_material">
@@ -305,5 +295,5 @@
       <origin xyz="0 0 0" rpy="0 -0 0"/>
       <geometry>
-        <mesh filename="final_assemble_rover_description/meshesbase_link__16.stl"/>
+        <mesh filename="package://assets/base_link__16.stl"/>
       </geometry>
     </collision>
@@ -312,5 +302,5 @@
       <origin xyz="0 0 0" rpy="0 -0 0"/>
       <geometry>
-        <mesh filename="final_assemble_rover_description/meshesbase_link__17.stl"/>
+        <mesh filename="package://assets/base_link__17.stl"/>
       </geometry>
       <material name="base_link_17_material">
@@ -321,5 +311,5 @@
       <origin xyz="0 0 0" rpy="0 -0 0"/>
       <geometry>
-        <mesh filename="final_assemble_rover_description/meshesbase_link__17.stl"/>
+        <mesh filename="package://assets/base_link__17.stl"/>
       </geometry>
     </collision>
@@ -328,5 +318,5 @@
       <origin xyz="0 0 0" rpy="0 -0 0"/>
       <geometry>
-        <mesh filename="final_assemble_rover_description/meshesbase_link__18.stl"/>
+        <mesh filename="package://assets/base_link__18.stl"/>
       </geometry>
       <material name="base_link_18_material">
@@ -337,5 +327,5 @@
       <origin xyz="0 0 0" rpy="0 -0 0"/>
       <geometry>
-        <mesh filename="final_assemble_rover_description/meshesbase_link__18.stl"/>
+        <mesh filename="package://assets/base_link__18.stl"/>
       </geometry>
     </collision>
@@ -344,5 +334,5 @@
       <origin xyz="0 0 0" rpy="0 -0 0"/>
       <geometry>
-        <mesh filename="final_assemble_rover_description/meshesbase_link__19.stl"/>
+        <mesh filename="package://assets/base_link__19.stl"/>
       </geometry>
       <material name="base_link_19_material">
@@ -353,5 +343,5 @@
       <origin xyz="0 0 0" rpy="0 -0 0"/>
       <geometry>
-        <mesh filename="final_assemble_rover_description/meshesbase_link__19.stl"/>
+        <mesh filename="package://assets/base_link__19.stl"/>
       </geometry>
     </collision>
@@ -360,5 +350,5 @@
       <origin xyz="0 0 0" rpy="0 -0 0"/>
       <geometry>
-        <mesh filename="final_assemble_rover_description/meshesbase_link__20.stl"/>
+        <mesh filename="package://assets/base_link__20.stl"/>
       </geometry>
       <material name="base_link_20_material">
@@ -369,5 +359,5 @@
       <origin xyz="0 0 0" rpy="0 -0 0"/>
       <geometry>
-        <mesh filename="final_assemble_rover_description/meshesbase_link__20.stl"/>
+        <mesh filename="package://assets/base_link__20.stl"/>
       </geometry>
     </collision>
@@ -376,5 +366,5 @@
       <origin xyz="0 0 0" rpy="0 -0 0"/>
       <geometry>
-        <mesh filename="final_assemble_rover_description/meshesbase_link__21.stl"/>
+        <mesh filename="package://assets/base_link__21.stl"/>
       </geometry>
       <material name="base_link_21_material">
@@ -385,5 +375,5 @@
       <origin xyz="0 0 0" rpy="0 -0 0"/>
       <geometry>
-        <mesh filename="final_assemble_rover_description/meshesbase_link__21.stl"/>
+        <mesh filename="package://assets/base_link__21.stl"/>
       </geometry>
     </collision>
@@ -392,5 +382,5 @@
       <origin xyz="0 0 0" rpy="0 -0 0"/>
       <geometry>
-        <mesh filename="final_assemble_rover_description/meshesbase_link__22.stl"/>
+        <mesh filename="package://assets/base_link__22.stl"/>
       </geometry>
       <material name="base_link_22_material">
@@ -401,5 +391,5 @@
       <origin xyz="0 0 0" rpy="0 -0 0"/>
       <geometry>
-        <mesh filename="final_assemble_rover_description/meshesbase_link__22.stl"/>
+        <mesh filename="package://assets/base_link__22.stl"/>
       </geometry>
     </collision>
@@ -408,5 +398,5 @@
       <origin xyz="0 0 0" rpy="0 -0 0"/>
       <geometry>
-        <mesh filename="final_assemble_rover_description/meshesbase_link__23.stl"/>
+        <mesh filename="package://assets/base_link__23.stl"/>
       </geometry>
       <material name="base_link_23_material">
@@ -417,5 +407,5 @@
       <origin xyz="0 0 0" rpy="0 -0 0"/>
       <geometry>
-        <mesh filename="final_assemble_rover_description/meshesbase_link__23.stl"/>
+        <mesh filename="package://assets/base_link__23.stl"/>
       </geometry>
     </collision>
@@ -424,5 +414,5 @@
       <origin xyz="0 0 0" rpy="0 -0 0"/>
       <geometry>
-        <mesh filename="final_assemble_rover_description/meshesbase_link__24.stl"/>
+        <mesh filename="package://assets/base_link__24.stl"/>
       </geometry>
       <material name="base_link_24_material">
@@ -433,5 +423,5 @@
       <origin xyz="0 0 0" rpy="0 -0 0"/>
       <geometry>
-        <mesh filename="final_assemble_rover_description/meshesbase_link__24.stl"/>
+        <mesh filename="package://assets/base_link__24.stl"/>
       </geometry>
     </collision>
@@ -440,5 +430,5 @@
       <origin xyz="0 0 0" rpy="0 -0 0"/>
       <geometry>
-        <mesh filename="final_assemble_rover_description/mesheslaser_link_1_1__3.stl"/>
+        <mesh filename="package://assets/laser_link_1_1__3.stl"/>
       </geometry>
       <material name="laser_link_1_1_3_material">
@@ -449,5 +439,5 @@
       <origin xyz="0 0 0" rpy="0 -0 0"/>
       <geometry>
-        <mesh filename="final_assemble_rover_description/mesheslaser_link_1_1__3.stl"/>
+        <mesh filename="package://assets/laser_link_1_1__3.stl"/>
       </geometry>
     </collision>
@@ -456,5 +446,5 @@
       <origin xyz="0 0 0" rpy="0 -0 0"/>
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