Commit message: assembly

File: final_assemble_rover_description/urdf/final_assemble_rover.xacro (robot description, xacro)
@@ -14,5 +14,5 @@
       <origin xyz="0 0 0" rpy="0 -0 0"/>
       <geometry>
-        <mesh filename="package://assets/base_link.stl"/>
+        <mesh filename="final_assemble_rover_description/meshesbase_link.stl"/>
       </geometry>
       <material name="base_link_material">
@@ -23,5 +23,5 @@
       <origin xyz="0 0 0" rpy="0 -0 0"/>
       <geometry>
-        <mesh filename="package://assets/base_link.stl"/>
+        <mesh filename="final_assemble_rover_description/meshesbase_link.stl"/>
       </geometry>
     </collision>
@@ -30,5 +30,5 @@
       <origin xyz="0 0 0" rpy="0 -0 0"/>
       <geometry>
-        <mesh filename="package://assets/base_link__2.stl"/>
+        <mesh filename="final_assemble_rover_description/meshesbase_link__2.stl"/>
       </geometry>
       <material name="base_link_2_material">
@@ -39,5 +39,5 @@
       <origin xyz="0 0 0" rpy="0 -0 0"/>
       <geometry>
-        <mesh filename="package://assets/base_link__2.stl"/>
+        <mesh filename="final_assemble_rover_description/meshesbase_link__2.stl"/>
       </geometry>
     </collision>
@@ -46,5 +46,5 @@
       <origin xyz="0 0 0" rpy="0 -0 0"/>
       <geometry>
-        <mesh filename="package://assets/base_link__3.stl"/>
+        <mesh filename="final_assemble_rover_description/meshesbase_link__3.stl"/>
       </geometry>
       <material name="base_link_3_material">
@@ -55,5 +55,5 @@
       <origin xyz="0 0 0" rpy="0 -0 0"/>
       <geometry>
-        <mesh filename="package://assets/base_link__3.stl"/>
+        <mesh filename="final_assemble_rover_description/meshesbase_link__3.stl"/>
       </geometry>
     </collision>
@@ -62,5 +62,5 @@
       <origin xyz="0 0 0" rpy="0 -0 0"/>
       <geometry>
-        <mesh filename="package://assets/laser_link_1_1.stl"/>
+        <mesh filename="final_assemble_rover_description/mesheslaser_link_1_1.stl"/>
       </geometry>
       <material name="laser_link_1_1_material">
@@ -71,5 +71,5 @@
       <origin xyz="0 0 0" rpy="0 -0 0"/>
       <geometry>
-        <mesh filename="package://assets/laser_link_1_1.stl"/>
+        <mesh filename="final_assemble_rover_description/mesheslaser_link_1_1.stl"/>
       </geometry>
     </collision>
@@ -78,5 +78,5 @@
       <origin xyz="0 0 0" rpy="0 -0 0"/>
       <geometry>
-        <mesh filename="package://assets/base_link__4.stl"/>
+        <mesh filename="final_assemble_rover_description/meshesbase_link__4.stl"/>
       </geometry>
       <material name="base_link_4_material">
@@ -87,5 +87,5 @@
       <origin xyz="0 0 0" rpy="0 -0 0"/>
       <geometry>
-        <mesh filename="package://assets/base_link__4.stl"/>
+        <mesh filename="final_assemble_rover_description/meshesbase_link__4.stl"/>
       </geometry>
     </collision>
@@ -94,5 +94,5 @@
       <origin xyz="0 0 0" rpy="0 -0 0"/>
       <geometry>
-        <mesh filename="package://assets/base_link__5.stl"/>
+        <mesh filename="final_assemble_rover_description/meshesbase_link__5.stl"/>
       </geometry>
       <material name="base_link_5_material">
@@ -103,5 +103,5 @@
       <origin xyz="0 0 0" rpy="0 -0 0"/>
       <geometry>
-        <mesh filename="package://assets/base_link__5.stl"/>
+        <mesh filename="final_assemble_rover_description/meshesbase_link__5.stl"/>
       </geometry>
     </collision>
@@ -110,5 +110,5 @@
       <origin xyz="0 0 0" rpy="0 -0 0"/>
       <geometry>
-        <mesh filename="package://assets/base_link__6.stl"/>
+        <mesh filename="final_assemble_rover_description/meshesbase_link__6.stl"/>
       </geometry>
       <material name="base_link_6_material">
@@ -119,5 +119,5 @@
       <origin xyz="0 0 0" rpy="0 -0 0"/>
       <geometry>
-        <mesh filename="package://assets/base_link__6.stl"/>
+        <mesh filename="final_assemble_rover_description/meshesbase_link__6.stl"/>
       </geometry>
     </collision>
@@ -126,5 +126,5 @@
       <origin xyz="0 0 0" rpy="0 -0 0"/>
       <geometry>
-        <mesh filename="package://assets/base_link__7.stl"/>
+        <mesh filename="final_assemble_rover_description/meshesbase_link__7.stl"/>
       </geometry>
       <material name="base_link_7_material">
@@ -135,5 +135,5 @@
       <origin xyz="0 0 0" rpy="0 -0 0"/>
       <geometry>
-        <mesh filename="package://assets/base_link__7.stl"/>
+        <mesh filename="final_assemble_rover_description/meshesbase_link__7.stl"/>
       </geometry>
     </collision>
@@ -142,5 +142,5 @@
       <origin xyz="0 0 0" rpy="0 -0 0"/>
       <geometry>
-        <mesh filename="package://assets/base_link__8.stl"/>
+        <mesh filename="final_assemble_rover_description/meshesbase_link__8.stl"/>
       </geometry>
       <material name="base_link_8_material">
@@ -151,5 +151,5 @@
       <origin xyz="0 0 0" rpy="0 -0 0"/>
       <geometry>
-        <mesh filename="package://assets/base_link__8.stl"/>
+        <mesh filename="final_assemble_rover_description/meshesbase_link__8.stl"/>
       </geometry>
     </collision>
@@ -158,5 +158,5 @@
       <origin xyz="0 0 0" rpy="0 -0 0"/>
       <geometry>
-        <mesh filename="package://assets/base_link__9.stl"/>
+        <mesh filename="final_assemble_rover_description/meshesbase_link__9.stl"/>
       </geometry>
       <material name="base_link_9_material">
@@ -167,5 +167,5 @@
       <origin xyz="0 0 0" rpy="0 -0 0"/>
       <geometry>
-        <mesh filename="package://assets/base_link__9.stl"/>
+        <mesh filename="final_assemble_rover_description/meshesbase_link__9.stl"/>
       </geometry>
     </collision>
@@ -174,5 +174,5 @@
       <origin xyz="0 0 0" rpy="0 -0 0"/>
       <geometry>
-        <mesh filename="package://assets/base_link__10.stl"/>
+        <mesh filename="final_assemble_rover_description/meshesbase_link__10.stl"/>
       </geometry>
       <material name="base_link_10_material">
@@ -183,5 +183,5 @@
       <origin xyz="0 0 0" rpy="0 -0 0"/>
       <geometry>
-        <mesh filename="package://assets/base_link__10.stl"/>
+        <mesh filename="final_assemble_rover_description/meshesbase_link__10.stl"/>
       </geometry>
     </collision>
@@ -190,5 +190,5 @@
       <origin xyz="0 0 0" rpy="0 -0 0"/>
       <geometry>
-        <mesh filename="package://assets/base_link__11.stl"/>
+        <mesh filename="final_assemble_rover_description/meshesbase_link__11.stl"/>
       </geometry>
       <material name="base_link_11_material">
@@ -199,5 +199,5 @@
       <origin xyz="0 0 0" rpy="0 -0 0"/>
       <geometry>
-        <mesh filename="package://assets/base_link__11.stl"/>
+        <mesh filename="final_assemble_rover_description/meshesbase_link__11.stl"/>
       </geometry>
     </collision>
@@ -206,5 +206,5 @@
       <origin xyz="0 0 0" rpy="0 -0 0"/>
       <geometry>
-        <mesh filename="package://assets/base_link__12.stl"/>
+        <mesh filename="final_assemble_rover_description/meshesbase_link__12.stl"/>
       </geometry>
       <material name="base_link_12_material">
@@ -215,5 +215,5 @@
       <origin xyz="0 0 0" rpy="0 -0 0"/>
       <geometry>
-        <mesh filename="package://assets/base_link__12.stl"/>
+        <mesh filename="final_assemble_rover_description/meshesbase_link__12.stl"/>
       </geometry>
     </collision>
@@ -222,5 +222,5 @@
       <origin xyz="0 0 0" rpy="0 -0 0"/>
       <geometry>
-        <mesh filename="package://assets/base_link__13.stl"/>
+        <mesh filename="final_assemble_rover_description/meshesbase_link__13.stl"/>
       </geometry>
       <material name="base_link_13_material">
@@ -231,5 +231,5 @@
       <origin xyz="0 0 0" rpy="0 -0 0"/>
       <geometry>
-        <mesh filename="package://assets/base_link__13.stl"/>
+        <mesh filename="final_assemble_rover_description/meshesbase_link__13.stl"/>
       </geometry>
     </collision>
@@ -238,5 +238,5 @@
       <origin xyz="0 0 0" rpy="0 -0 0"/>
       <geometry>
-        <mesh filename="package://assets/base_link__14.stl"/>
+        <mesh filename="final_assemble_rover_description/meshesbase_link__14.stl"/>
       </geometry>
       <material name="base_link_14_material">
@@ -247,5 +247,5 @@
       <origin xyz="0 0 0" rpy="0 -0 0"/>
       <geometry>
-        <mesh filename="package://assets/base_link__14.stl"/>
+        <mesh filename="final_assemble_rover_description/meshesbase_link__14.stl"/>
       </geometry>
     </collision>
@@ -254,5 +254,5 @@
       <origin xyz="0 0 0" rpy="0 -0 0"/>
       <geometry>
-        <mesh filename="package://assets/base_link__15.stl"/>
+        <mesh filename="final_assemble_rover_description/meshesbase_link__15.stl"/>
       </geometry>
       <material name="base_link_15_material">
@@ -263,5 +263,5 @@
       <origin xyz="0 0 0" rpy="0 -0 0"/>
       <geometry>
-        <mesh filename="package://assets/base_link__15.stl"/>
+        <mesh filename="final_assemble_rover_description/meshesbase_link__15.stl"/>
       </geometry>
     </collision>
@@ -270,5 +270,5 @@
       <origin xyz="0 0 0" rpy="0 -0 0"/>
       <geometry>
-        <mesh filename="package://assets/laser_link_1_1__2.stl"/>
+        <mesh filename="final_assemble_rover_description/mesheslaser_link_1_1__2.stl"/>
       </geometry>
       <material name="laser_link_1_1_2_material">
@@ -279,5 +279,5 @@
       <origin xyz="0 0 0" rpy="0 -0 0"/>
       <geometry>
-        <mesh filename="package://assets/laser_link_1_1__2.stl"/>
+        <mesh filename="final_assemble_rover_description/mesheslaser_link_1_1__2.stl"/>
       </geometry>
     </collision>
@@ -286,5 +286,5 @@
       <origin xyz="0 0 0" rpy="0 -0 0"/>
       <geometry>
-        <mesh filename="package://assets/base_link__16.stl"/>
+        <mesh filename="final_assemble_rover_description/meshesbase_link__16.stl"/>
       </geometry>
       <material name="base_link_16_material">
@@ -295,5 +295,5 @@
       <origin xyz="0 0 0" rpy="0 -0 0"/>
       <geometry>
-        <mesh filename="package://assets/base_link__16.stl"/>
+        <mesh filename="final_assemble_rover_description/meshesbase_link__16.stl"/>
       </geometry>
     </collision>
@@ -302,5 +302,5 @@
       <origin xyz="0 0 0" rpy="0 -0 0"/>
       <geometry>
-        <mesh filename="package://assets/base_link__17.stl"/>
+        <mesh filename="final_assemble_rover_description/meshesbase_link__17.stl"/>
       </geometry>
       <material name="base_link_17_material">
@@ -311,5 +311,5 @@
       <origin xyz="0 0 0" rpy="0 -0 0"/>
       <geometry>
-        <mesh filename="package://assets/base_link__17.stl"/>
+        <mesh filename="final_assemble_rover_description/meshesbase_link__17.stl"/>
       </geometry>
     </collision>
@@ -318,5 +318,5 @@
       <origin xyz="0 0 0" rpy="0 -0 0"/>
       <geometry>
-        <mesh filename="package://assets/base_link__18.stl"/>
+        <mesh filename="final_assemble_rover_description/meshesbase_link__18.stl"/>
       </geometry>
       <material name="base_link_18_material">
@@ -327,5 +327,5 @@
       <origin xyz="0 0 0" rpy="0 -0 0"/>
       <geometry>
-        <mesh filename="package://assets/base_link__18.stl"/>
+        <mesh filename="final_assemble_rover_description/meshesbase_link__18.stl"/>
       </geometry>
     </collision>
@@ -334,5 +334,5 @@
       <origin xyz="0 0 0" rpy="0 -0 0"/>
       <geometry>
-        <mesh filename="package://assets/base_link__19.stl"/>
+        <mesh filename="final_assemble_rover_description/meshesbase_link__19.stl"/>
       </geometry>
       <material name="base_link_19_material">
@@ -343,5 +343,5 @@
       <origin xyz="0 0 0" rpy="0 -0 0"/>
       <geometry>
-        <mesh filename="package://assets/base_link__19.stl"/>
+        <mesh filename="final_assemble_rover_description/meshesbase_link__19.stl"/>
       </geometry>
     </collision>
@@ -350,5 +350,5 @@
       <origin xyz="0 0 0" rpy="0 -0 0"/>
       <geometry>
-        <mesh filename="package://assets/base_link__20.stl"/>
+        <mesh filename="final_assemble_rover_description/meshesbase_link__20.stl"/>
       </geometry>
       <material name="base_link_20_material">
@@ -359,5 +359,5 @@
       <origin xyz="0 0 0" rpy="0 -0 0"/>
       <geometry>
-        <mesh filename="package://assets/base_link__20.stl"/>
+        <mesh filename="final_assemble_rover_description/meshesbase_link__20.stl"/>
       </geometry>
     </collision>
@@ -366,5 +366,5 @@
       <origin xyz="0 0 0" rpy="0 -0 0"/>
       <geometry>
-        <mesh filename="package://assets/base_link__21.stl"/>
+        <mesh filename="final_assemble_rover_description/meshesbase_link__21.stl"/>
       </geometry>
       <material name="base_link_21_material">
@@ -375,5 +375,5 @@
       <origin xyz="0 0 0" rpy="0 -0 0"/>
       <geometry>
-        <mesh filename="package://assets/base_link__21.stl"/>
+        <mesh filename="final_assemble_rover_description/meshesbase_link__21.stl"/>
       </geometry>
     </collision>
@@ -382,5 +382,5 @@
       <origin xyz="0 0 0" rpy="0 -0 0"/>
       <geometry>
-        <mesh filename="package://assets/base_link__22.stl"/>
+        <mesh filename="final_assemble_rover_description/meshesbase_link__22.stl"/>
       </geometry>
       <material name="base_link_22_material">
@@ -391,5 +391,5 @@
       <origin xyz="0 0 0" rpy="0 -0 0"/>
       <geometry>
-        <mesh filename="package://assets/base_link__22.stl"/>
+        <mesh filename="final_assemble_rover_description/meshesbase_link__22.stl"/>
       </geometry>
     </collision>
@@ -398,5 +398,5 @@
       <origin xyz="0 0 0" rpy="0 -0 0"/>
       <geometry>
-        <mesh filename="package://assets/base_link__23.stl"/>
+        <mesh filename="final_assemble_rover_description/meshesbase_link__23.stl"/>
       </geometry>
       <material name="base_link_23_material">
@@ -407,5 +407,5 @@
       <origin xyz="0 0 0" rpy="0 -0 0"/>
       <geometry>
-        <mesh filename="package://assets/base_link__23.stl"/>
+        <mesh filename="final_assemble_rover_description/meshesbase_link__23.stl"/>
       </geometry>
     </collision>
@@ -414,5 +414,5 @@
       <origin xyz="0 0 0" rpy="0 -0 0"/>
       <geometry>
-        <mesh filename="package://assets/base_link__24.stl"/>
+        <mesh filename="final_assemble_rover_description/meshesbase_link__24.stl"/>
       </geometry>
       <material name="base_link_24_material">
@@ -423,5 +423,5 @@
       <origin xyz="0 0 0" rpy="0 -0 0"/>
       <geometry>
-        <mesh filename="package://assets/base_link__24.stl"/>
+        <mesh filename="final_assemble_rover_description/meshesbase_link__24.stl"/>
       </geometry>
     </collision>
@@ -430,5 +430,5 @@
       <origin xyz="0 0 0" rpy="0 -0 0"/>
       <geometry>
-        <mesh filename="package://assets/laser_link_1_1__3.stl"/>
+        <mesh filename="final_assemble_rover_description/mesheslaser_link_1_1__3.stl"/>
       </geometry>
       <material name="laser_link_1_1_3_material">
@@ -439,5 +439,5 @@
       <origin xyz="0 0 0" rpy="0 -0 0"/>
       <geometry>
-        <mesh filename="package://assets/laser_link_1_1__3.stl"/>
+        <mesh filename="final_assemble_rover_description/mesheslaser_link_1_1__3.stl"/>
       </geometry>
     </collision>
@@ -446,5 +446,5 @@
       <origin xyz="0 0 0" rpy="0 -0 0"/>
       <geometry>
-        <mesh filename="package://assets/base_link__25.stl"/>
+        <mesh filename="final_assemble_rover_description/meshesbase_link__25.stl"/>
       </geometry>
       <material name="base_link_25_material">
@@ -455,5 +455,5 @@
       <origin xyz="0 0 0" rpy="0 -0 0"/>
       <geometry>
-        <mesh filename="package://assets/base_link__25.stl"/>
+        <mesh filename="final_assemble_rover_description/meshesbase_link__25.stl"/>
       </geometry>
     </collision>
@@ -462,5 +462,5 @@
       <origin xyz="0 0 0" rpy="0 -0 0"/>
       <geometry>
-        <mesh filename="package://assets/base_link__26.stl"/>
+        <mesh filename="final_assemble_rover_description/meshesbase_link__26.stl"/>
       </geometry>
       <material name="base_link_26_material">
@@ -471,5 +471,5 @@
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
Commit message: check add

File: final_assemble_rover_description/urdf/final_assemble_rover.xacro (robot description, xacro)
@@ -6606,5 +6606,5 @@
   </link>
   <!-- Joint from base_link to castor_link_1_1 -->
-  <joint name="castor_joint" type="ball">
+  <joint name="castor_joint" type="fixed">
     <origin xyz="0.0397465 0 -0.0076" rpy="-1.67306 -0.644916 1.42189"/>
     <parent link="base_link"/>

Commit message: update

File: final_assemble_rover_description/urdf/final_assemble_rover.xacro (robot description, xacro)
@@ -17,6 +17,6 @@
     <inertial>
       <origin xyz="-0.00490882 -0.000846201 0.0714046" rpy="0 0 0"/>
-      <mass value="0.222325"/>
-      <inertia ixx="0.00059991" ixy="-8.12726e-07" ixz="-3.66324e-05" iyy="0.000620644" iyz="-1.74055e-06" izz="0.00031087"/>
+      <mass value="1.0"/>
+      <inertia ixx="0.1" ixy="0.0" ixz="0.0" iyy="0.1" iyz="0.0" izz="0.1"/>
     </inertial>
     <!-- Part base_link -->
@@ -6521,6 +6521,6 @@
     <inertial>
       <origin xyz="2.4435e-08 2.83911e-07 -0.01589" rpy="0 0 0"/>
-      <mass value="0.0327076"/>
-      <inertia ixx="1.35205e-05" ixy="-6.6e-11" ixz="8e-12" iyy="1.35201e-05" iyz="9.8e-11" izz="2.24167e-05"/>
+      <mass value="1.0"/>
+      <inertia ixx="0.1" ixy="0.0" ixz="0.0" iyy="0.1" iyz="0.0" izz="0.1"/>
     </inertial>
     <!-- Part right_wheel_link_1_1 -->
@@ -6553,6 +6553,6 @@
     <inertial>
       <origin xyz="-2.74849e-07 7.5237e-08 -0.01589" rpy="0 0 0"/>
-      <mass value="0.0327076"/>
-      <inertia ixx="1.35202e-05" ixy="1.27e-10" ixz="-9.5e-11" iyy="1.35205e-05" iyz="2.6e-11" izz="2.24167e-05"/>
+      <mass value="1.0"/>
+      <inertia ixx="0.1" ixy="0.0" ixz="0.0" iyy="0.1" iyz="0.0" izz="0.1"/>
     </inertial>
     <!-- Part left_wheel_link_1_1 -->
@@ -6585,6 +6585,6 @@
     <inertial>
       <origin xyz="0 0 0" rpy="0 0 0"/>
-      <mass value="0.00387924"/>
-      <inertia ixx="7.6033e-08" ixy="0" ixz="-0" iyy="7.6033e-08" iyz="-0" izz="7.6033e-08"/>
+      <mass value="1.0"/>
+      <inertia ixx="0.1" ixy="0.0" ixz="0.0" iyy="0.1" iyz="0.0" izz="0.1"/>
     </inertial>
     <!-- Part castor_link_1_1 -->
