Commit message: final_assemble

File: final_assemble_rover_description/urdf/final_assemble_rover.xacro (robot description, xacro)
@@ -1,5 +1,5 @@
 <?xml version="1.0"?>
 <robot xmlns:xacro="http://www.ros.org/wiki/xacro" name="final_assemble_rover">
-    <!-- INERTIA MACROS (To prevent the Gazebo physics explosions) -->
+    <!-- INERTIA MAPPING MACROS -->
     <xacro:macro name="box_inertia" params="m w h d">
         <inertial>
@@ -20,7 +20,14 @@
         </inertial>
     </xacro:macro>
-    <!-- BASE FOOTPRINT (Ground Level) -->
+    <!-- MATERIAL COLOR DEFINITIONS (For RViz View) -->
+    <material name="red"><color rgba="0.8 0.1 0.1 1.0"/></material>
+    <material name="black"><color rgba="0.1 0.1 0.1 1.0"/></material>
+    <material name="yellow"><color rgba="0.9 0.7 0.0 1.0"/></material>
+    <material name="silver"><color rgba="0.75 0.75 0.75 1.0"/></material>
+    <material name="grey"><color rgba="0.3 0.3 0.3 1.0"/></material>
+    <material name="white"><color rgba="0.9 0.9 0.9 1.0"/></material>
+    <!-- BASE FOOTPRINT (Projected Ground Origin) -->
     <link name="base_footprint"/>
-    <!-- CHASSIS (12cm x 11cm x 5cm) -->
+    <!-- MAIN LOWER CHASSIS ASSEMBLY -->
     <joint name="base_joint" type="fixed">
         <parent link="base_footprint"/>
@@ -29,9 +36,34 @@
     </joint>
     <link name="base_link">
+        <!-- Main Red Box Body (12x11x5 cm) -->
         <visual>
             <geometry>
                 <box size="0.12 0.11 0.05"/>
             </geometry>
-            <material name="red"><color rgba="0.8 0.1 0.1 1.0"/></material>
+            <material name="red"/>
+        </visual>
+        <!-- Front Left Standoff Pillar -->
+        <visual>
+            <origin xyz="0.04 0.045 0.05" rpy="0 0 0"/>
+            <geometry><cylinder radius="0.004" length="0.05"/></geometry>
+            <material name="silver"/>
+        </visual>
+        <!-- Front Right Standoff Pillar -->
+        <visual>
+            <origin xyz="0.04 -0.045 0.05" rpy="0 0 0"/>
+            <geometry><cylinder radius="0.004" length="0.05"/></geometry>
+            <material name="silver"/>
+        </visual>
+        <!-- Rear Left Standoff Pillar -->
+        <visual>
+            <origin xyz="-0.04 0.045 0.05" rpy="0 0 0"/>
+            <geometry><cylinder radius="0.004" length="0.05"/></geometry>
+            <material name="silver"/>
+        </visual>
+        <!-- Rear Right Standoff Pillar -->
+        <visual>
+            <origin xyz="-0.04 -0.045 0.05" rpy="0 0 0"/>
+            <geometry><cylinder radius="0.004" length="0.05"/></geometry>
+            <material name="silver"/>
         </visual>
         <collision>
@@ -40,110 +72,134 @@
             </geometry>
         </collision>
-        <xacro:box_inertia m="1.0" w="0.12" h="0.11" d="0.05"/>
-    </link>
+        <xacro:box_inertia m="1.2" w="0.12" h="0.11" d="0.05"/>
+    </link>
+    <!-- Gazebo Color Overrides for Chassis Links -->
     <gazebo reference="base_link"><material>Gazebo/Red</material></gazebo>
-    <!-- LEFT WHEEL (Radius 3cm, Width 2.5cm) -->
+    <!-- MID-TIER ELECTRONICS DECK -->
+    <joint name="mid_deck_joint" type="fixed">
+        <parent link="base_link"/>
+        <child link="mid_deck_link"/>
+        <origin xyz="0 0 0.075" rpy="0 0 0"/>
+    </joint>
+    <link name="mid_deck_link">
+        <visual>
+            <geometry>
+                <box size="0.12 0.11 0.004"/>
+            </geometry>
+            <material name="grey"/>
+        </visual>
+        <collision>
+            <geometry>
+                <box size="0.12 0.11 0.004"/>
+            </geometry>
+        </collision>
+        <xacro:box_inertia m="0.2" w="0.12" h="0.11" d="0.004"/>
+    </link>
+    <gazebo reference="mid_deck_link"><material>Gazebo/Grey</material></gazebo>
+    <!-- LEFT DRIVE WHEEL (Black Tread + Concentric Yellow Rim Hub) -->
     <joint name="left_wheel_joint" type="continuous">
         <parent link="base_link"/>
         <child link="left_wheel"/>
-        <origin xyz="-0.035 0.0675 -0.025" rpy="-1.5708 0 0"/>
+        <origin xyz="-0.035 0.068 -0.025" rpy="-1.5708 0 0"/>
         <axis xyz="0 0 1"/>
     </joint>
     <link name="left_wheel">
-        <visual>
-            <geometry>
-                <cylinder radius="0.03" length="0.025"/>
-            </geometry>
-            <material name="black"><color rgba="0.1 0.1 0.1 1.0"/></material>
-        </visual>
-        <collision>
-            <geometry>
-                <cylinder radius="0.03" length="0.025"/>
-            </geometry>
-        </collision>
-        <xacro:cylinder_inertia m="0.2" r="0.03" h="0.025"/>
-    </link>
-    <gazebo reference="left_wheel"><material>Gazebo/Black</material></gazebo>
-    <!-- RIGHT WHEEL (Radius 3cm, Width 2.5cm) -->
+        <!-- Outer Rubber Tire -->
+        <visual>
+            <geometry><cylinder radius="0.03" length="0.025"/></geometry>
+            <material name="black"/>
+        </visual>
+        <!-- Inner Gold/Yellow Hub Core -->
+        <visual>
+            <origin xyz="0 0 0.001" rpy="0 0 0"/>
+            <geometry><cylinder radius="0.022" length="0.024"/></geometry>
+            <material name="yellow"/>
+        </visual>
+        <collision>
+            <geometry><cylinder radius="0.03" length="0.025"/></geometry>
+        </collision>
+        <xacro:cylinder_inertia m="0.25" r="0.03" h="0.025"/>
+    </link>
+    <gazebo reference="left_wheel"><material>Gazebo/DarkGrey</material></gazebo>
+    <!-- RIGHT DRIVE WHEEL (Black Tread + Concentric Yellow Rim Hub) -->
     <joint name="right_wheel_joint" type="continuous">
         <parent link="base_link"/>
         <child link="right_wheel"/>
-        <origin xyz="-0.035 -0.0675 -0.025" rpy="1.5708 0 0"/>
+        <origin xyz="-0.035 -0.068 -0.025" rpy="1.5708 0 0"/>
         <axis xyz="0 0 -1"/>
     </joint>
     <link name="right_wheel">
-        <visual>
-            <geometry>
-                <cylinder radius="0.03" length="0.025"/>
-            </geometry>
+        <!-- Outer Rubber Tire -->
+        <visual>
+            <geometry><cylinder radius="0.03" length="0.025"/></geometry>
             <material name="black"/>
         </visual>
-        <collision>
-            <geometry>
-                <cylinder radius="0.03" length="0.025"/>
-            </geometry>
-        </collision>
-        <xacro:cylinder_inertia m="0.2" r="0.03" h="0.025"/>
-    </link>
-    <gazebo reference="right_wheel"><material>Gazebo/Black</material></gazebo>
-    <!-- CASTOR WHEEL (Radius 2cm) -->
+        <!-- Inner Gold/Yellow Hub Core -->
+        <visual>
+            <origin xyz="0 0 0.001" rpy="0 0 0"/>
+            <geometry><cylinder radius="0.022" length="0.024"/></geometry>
+            <material name="yellow"/>
+        </visual>
+        <collision>
+            <geometry><cylinder radius="0.03" length="0.025"/></geometry>
+        </collision>
+        <xacro:cylinder_inertia m="0.25" r="0.03" h="0.025"/>
+    </link>
+    <gazebo reference="right_wheel"><material>Gazebo/DarkGrey</material></gazebo>
+    <!-- BALANCING CASTER ASSEMBLY -->
     <joint name="castor_joint" type="fixed">
         <parent link="base_link"/>
         <child link="castor_wheel"/>
-        <origin xyz="0.04 0 -0.035" rpy="0 0 0"/>
+        <origin xyz="0.045 0 -0.035" rpy="0 0 0"/>
     </joint>
     <link name="castor_wheel">
         <visual>
-            <geometry>
-                <sphere radius="0.02"/>
-            </geometry>
-            <material name="white"><color rgba="0.9 0.9 0.9 1.0"/></material>
-        </visual>
-        <collision>
-            <geometry>
-                <sphere radius="0.02"/>
-            </geometry>
+            <geometry><sphere radius="0.02"/></geometry>
+            <material name="white"/>
+        </visual>
+        <collision>
+            <geometry><sphere radius="0.02"/></geometry>
         </collision>
         <xacro:sphere_inertia m="0.1" r="0.02"/>
     </link>
-    <!-- ZERO FRICTION TAG: Prevents castor from dragging in Gazebo -->
     <gazebo reference="castor_wheel">
         <material>Gazebo/White</material>
-        <mu1>0.001</mu1>
-        <mu2>0.001</mu2>
+        <mu1>0.0001</mu1>
+        <mu2>0.0001</mu2>
     </gazebo>
-    <!-- VIRTUAL LIDAR PUCK -->
+    <!-- TOP-MOUNTED VIRTUAL LIDAR PUCK -->
     <joint name="lidar_joint" type="fixed">
-        <parent link="base_link"/>
+        <parent link="mid_deck_link"/>
         <child link="lidar_link"/>
-        <origin xyz="0 0 0.045" rpy="0 0 0"/>
+        <origin xyz="0 0 0.022" rpy="0 0 0"/>
     </joint>
     <link name="lidar_link">
-        <visual>
-            <geometry>
-                <cylinder radius="0.03" length="0.04"/>
-            </geometry>
+        <!-- Core Rotating Scanner Head -->
+        <visual>
+            <geometry><cylinder radius="0.03" length="0.035"/></geometry>
             <material name="black"/>
         </visual>
-        <collision>
-            <geometry>
-                <cylinder radius="0.03" length="0.04"/>
-            </geometry>
-        </collision>
-        <xacro:cylinder_inertia m="0.1" r="0.03" h="0.04"/>
+        <!-- Optical Sensor Lens Embellishment -->
+        <visual>
+            <origin xyz="0.025 0 0.005" rpy="0 1.5708 0"/>
+            <geometry><cylinder radius="0.006" length="0.01"/></geometry>
+            <material name="grey"/>
+        </visual>
+        <collision>
+            <geometry><cylinder radius="0.03" length="0.035"/></geometry>
+        </collision>
+        <xacro:cylinder_inertia m="0.15" r="0.03" h="0.035"/>
     </link>
     <gazebo reference="lidar_link"><material>Gazebo/Black</material></gazebo>
-    <!-- GAZEBO DIFFERENTIAL DRIVE PLUGIN -->
+    <!-- GAZEBO KINEMATIC CONTROL PLUGIN (Differential Drive Configuration) -->
     <gazebo>
         <plugin name="diff_drive" filename="libgazebo_ros_diff_drive.so">
-            <ros>
-                <namespace>/</namespace>
-            </ros>
+            <ros><namespace>/</namespace></ros>
             <left_joint>left_wheel_joint</left_joint>
             <right_joint>right_wheel_joint</right_joint>
-            <wheel_separation>0.135</wheel_separation>
+            <wheel_separation>0.136</wheel_separation>
             <wheel_diameter>0.06</wheel_diameter>
-            <max_wheel_torque>20</max_wheel_torque>
-            <max_wheel_acceleration>1.0</max_wheel_acceleration>
+            <max_wheel_torque>15</max_wheel_torque>
+            <max_wheel_acceleration>1.5</max_wheel_acceleration>
             <publish_odom>true</publish_odom>
             <publish_odom_tf>true</publish_odom_tf>
@@ -153,5 +209,5 @@
         </plugin>
     </gazebo>
-    <!-- GAZEBO VIRTUAL LIDAR PLUGIN (Feeds map data to Nav2) -->
+    <!-- GAZEBO SENSOR PLUGIN (Virtual LiDAR Linkage for Navigation Tricking) -->
     <gazebo reference="lidar_link">
         <sensor type="ray" name="virtual_lidar">
@@ -169,13 +225,11 @@
                 </scan>
                 <range>
-                    <min>0.15</min>
-                    <max>12.0</max>
+                    <min>0.12</min>
+                    <max>10.0</max>
                     <resolution>0.01</resolution>
                 </range>
             </ray>
             <plugin name="scan" filename="libgazebo_ros_ray_sensor.so">
-                <ros>
-                    <remapping>~/out:=scan</remapping>
-                </ros>
+                <ros><remapping>~/out:=scan</remapping></ros>
                 <output_type>sensor_msgs/LaserScan</output_type>
                 <frame_name>lidar_link</frame_name>
