Commit message: check

File: final_assemble_rover_description/urdf/final_assemble_rover.xacro (robot description, xacro)
@@ -1,71 +1,50 @@
 <?xml version="1.0"?>
-<robot xmlns:xacro="http://www.ros.org/wiki/xacro" name="final_assemble_rover">
-    <!-- INERTIA MAPPING MACROS -->
+<robot xmlns:xacro="http://www.ros.org/wiki/xacro" name="my_rover">
+    <!-- ========================================================== -->
+    <!-- INERTIA MACROS (Baked in so you don't need extra files)    -->
+    <!-- ========================================================== -->
     <xacro:macro name="box_inertia" params="m w h d">
         <inertial>
+            <origin xyz="0 0 0" rpy="0 0 0"/>
             <mass value="${m}"/>
-            <inertia ixx="${(m/12) * (h*h + d*d)}" ixy="0.0" ixz="0.0" iyy="${(m/12) * (w*w + d*d)}" iyz="0.0" izz="${(m/12) * (w*w + h*h)}"/>
+            <inertia ixx="${(m/12) * (h*h + d*d)}" ixy="0.0" ixz="0.0"
+                     iyy="${(m/12) * (w*w + d*d)}" iyz="0.0"
+                     izz="${(m/12) * (w*w + h*h)}"/>
         </inertial>
     </xacro:macro>
     <xacro:macro name="cylinder_inertia" params="m r h">
         <inertial>
+            <origin xyz="0 0 0" rpy="0 0 0"/>
             <mass value="${m}"/>
-            <inertia ixx="${(m/12) * (3*r*r + h*h)}" ixy="0.0" ixz="0.0" iyy="${(m/12) * (3*r*r + h*h)}" iyz="0.0" izz="${(m/2) * (r*r)}"/>
+            <inertia ixx="${(m/12) * (3*r*r + h*h)}" ixy="0" ixz="0"
+                     iyy="${(m/12) * (3*r*r + h*h)}" iyz="0"
+                     izz="${(m/2) * (r*r)}"/>
         </inertial>
     </xacro:macro>
     <xacro:macro name="sphere_inertia" params="m r">
         <inertial>
+            <origin xyz="0 0 0" rpy="0 0 0"/>
             <mass value="${m}"/>
-            <inertia ixx="${(2/5) * m * (r*r)}" ixy="0.0" ixz="0.0" iyy="${(2/5) * m * (r*r)}" iyz="0.0" izz="${(2/5) * m * (r*r)}"/>
+            <inertia ixx="${(2/5) * m * (r*r)}" ixy="0.0" ixz="0.0"
+                     iyy="${(2/5) * m * (r*r)}" iyz="0.0"
+                     izz="${(2/5) * m * (r*r)}"/>
         </inertial>
     </xacro:macro>
-    <!-- MATERIAL COLOR DEFINITIONS (For RViz View) -->
-    <material name="red"><color rgba="0.8 0.1 0.1 1.0"/></material>
-    <material name="black"><color rgba="0.1 0.1 0.1 1.0"/></material>
-    <material name="yellow"><color rgba="0.9 0.7 0.0 1.0"/></material>
-    <material name="silver"><color rgba="0.75 0.75 0.75 1.0"/></material>
-    <material name="grey"><color rgba="0.3 0.3 0.3 1.0"/></material>
-    <material name="white"><color rgba="0.9 0.9 0.9 1.0"/></material>
-    <!-- BASE FOOTPRINT (Projected Ground Origin) -->
-    <link name="base_footprint"/>
-    <!-- MAIN LOWER CHASSIS ASSEMBLY -->
-    <joint name="base_joint" type="fixed">
-        <parent link="base_footprint"/>
-        <child link="base_link"/>
-        <origin xyz="0 0 0.055" rpy="0 0 0"/>
-    </joint>
+    <!-- ========================================================== -->
+    <!-- ROBOT GEOMETRY & JOINTS                                    -->
+    <!-- ========================================================== -->
+    <!-- BASE LINK (Chassis) -->
     <link name="base_link">
-        <!-- Main Red Box Body (12x11x5 cm) -->
         <visual>
+            <origin xyz="0 0 0" rpy="0 0 0"/>
             <geometry>
-                <box size="0.12 0.11 0.05"/>
+                <mesh filename="file://$(find final_assemble_rover_description)/meshes/chasis.STL" scale="1 1 1"/>
             </geometry>
-            <material name="red"/>
-        </visual>
-        <!-- Front Left Standoff Pillar -->
-        <visual>
-            <origin xyz="0.04 0.045 0.05" rpy="0 0 0"/>
-            <geometry><cylinder radius="0.004" length="0.05"/></geometry>
-            <material name="silver"/>
-        </visual>
-        <!-- Front Right Standoff Pillar -->
-        <visual>
-            <origin xyz="0.04 -0.045 0.05" rpy="0 0 0"/>
-            <geometry><cylinder radius="0.004" length="0.05"/></geometry>
-            <material name="silver"/>
-        </visual>
-        <!-- Rear Left Standoff Pillar -->
-        <visual>
-            <origin xyz="-0.04 0.045 0.05" rpy="0 0 0"/>
-            <geometry><cylinder radius="0.004" length="0.05"/></geometry>
-            <material name="silver"/>
-        </visual>
-        <!-- Rear Right Standoff Pillar -->
-        <visual>
-            <origin xyz="-0.04 -0.045 0.05" rpy="0 0 0"/>
-            <geometry><cylinder radius="0.004" length="0.05"/></geometry>
-            <material name="silver"/>
+            <material name="red">
+                <color rgba="0.8 0.1 0.1 1.0"/>
+            </material>
         </visual>
         <collision>
+            <origin xyz="0 0 0" rpy="0 0 0"/>
             <geometry>
                 <box size="0.12 0.11 0.05"/>
@@ -74,166 +53,103 @@
         <xacro:box_inertia m="1.2" w="0.12" h="0.11" d="0.05"/>
     </link>
-    <!-- Gazebo Color Overrides for Chassis Links -->
-    <gazebo reference="base_link"><material>Gazebo/Red</material></gazebo>
-    <!-- MID-TIER ELECTRONICS DECK -->
-    <joint name="mid_deck_joint" type="fixed">
-        <parent link="base_link"/>
-        <child link="mid_deck_link"/>
-        <origin xyz="0 0 0.075" rpy="0 0 0"/>
-    </joint>
-    <link name="mid_deck_link">
-        <visual>
-            <geometry>
-                <box size="0.12 0.11 0.004"/>
-            </geometry>
-            <material name="grey"/>
-        </visual>
-        <collision>
-            <geometry>
-                <box size="0.12 0.11 0.004"/>
-            </geometry>
-        </collision>
-        <xacro:box_inertia m="0.2" w="0.12" h="0.11" d="0.004"/>
-    </link>
-    <gazebo reference="mid_deck_link"><material>Gazebo/Grey</material></gazebo>
-    <!-- LEFT DRIVE WHEEL (Black Tread + Concentric Yellow Rim Hub) -->
+    <!-- LEFT WHEEL -->
     <joint name="left_wheel_joint" type="continuous">
         <parent link="base_link"/>
         <child link="left_wheel"/>
-        <origin xyz="-0.035 0.068 -0.025" rpy="-1.5708 0 0"/>
+        <origin xyz="0.03 0.065 -0.02" rpy="-1.5708 0 0"/>
         <axis xyz="0 0 1"/>
     </joint>
     <link name="left_wheel">
-        <!-- Outer Rubber Tire -->
         <visual>
-            <geometry><cylinder radius="0.03" length="0.025"/></geometry>
-            <material name="black"/>
-        </visual>
-        <!-- Inner Gold/Yellow Hub Core -->
-        <visual>
-            <origin xyz="0 0 0.001" rpy="0 0 0"/>
-            <geometry><cylinder radius="0.022" length="0.024"/></geometry>
-            <material name="yellow"/>
+            <origin xyz="0 0 0" rpy="0 0 0"/>
+            <geometry>
+                <mesh filename="file://$(find final_assemble_rover_description)/meshes/wheel_link.STL" scale="1 1 1"/>
+            </geometry>
+            <material name="black">
+                <color rgba="0.1 0.1 0.1 1.0"/>
+            </material>
         </visual>
         <collision>
-            <geometry><cylinder radius="0.03" length="0.025"/></geometry>
+            <origin xyz="0 0 0" rpy="0 0 0"/>
+            <geometry>
+                <cylinder radius="0.03" length="0.025"/>
+            </geometry>
         </collision>
         <xacro:cylinder_inertia m="0.25" r="0.03" h="0.025"/>
     </link>
-    <gazebo reference="left_wheel"><material>Gazebo/DarkGrey</material></gazebo>
-    <!-- RIGHT DRIVE WHEEL (Black Tread + Concentric Yellow Rim Hub) -->
+    <!-- RIGHT WHEEL -->
     <joint name="right_wheel_joint" type="continuous">
         <parent link="base_link"/>
         <child link="right_wheel"/>
-        <origin xyz="-0.035 -0.068 -0.025" rpy="1.5708 0 0"/>
-        <axis xyz="0 0 -1"/>
+        <origin xyz="0.03 -0.065 -0.02" rpy="1.5708 0 0"/>
+        <axis xyz="0 0 1"/>
     </joint>
     <link name="right_wheel">
-        <!-- Outer Rubber Tire -->
         <visual>
-            <geometry><cylinder radius="0.03" length="0.025"/></geometry>
+            <origin xyz="0 0 0" rpy="0 0 0"/>
+            <geometry>
+                <mesh filename="file://$(find final_assemble_rover_description)/meshes/wheel_link.STL" scale="1 1 1"/>
+            </geometry>
             <material name="black"/>
         </visual>
-        <!-- Inner Gold/Yellow Hub Core -->
-        <visual>
-            <origin xyz="0 0 0.001" rpy="0 0 0"/>
-            <geometry><cylinder radius="0.022" length="0.024"/></geometry>
-            <material name="yellow"/>
-        </visual>
         <collision>
-            <geometry><cylinder radius="0.03" length="0.025"/></geometry>
+            <origin xyz="0 0 0" rpy="0 0 0"/>
+            <geometry>
+                <cylinder radius="0.03" length="0.025"/>
+            </geometry>
         </collision>
         <xacro:cylinder_inertia m="0.25" r="0.03" h="0.025"/>
     </link>
-    <gazebo reference="right_wheel"><material>Gazebo/DarkGrey</material></gazebo>
-    <!-- BALANCING CASTER ASSEMBLY -->
+    <!-- CASTOR BALL -->
     <joint name="castor_joint" type="fixed">
         <parent link="base_link"/>
-        <child link="castor_wheel"/>
-        <origin xyz="0.045 0 -0.035" rpy="0 0 0"/>
+        <child link="castor_link"/>
+        <origin xyz="-0.04 0 -0.03" rpy="0 0 0"/>
     </joint>
-    <link name="castor_wheel">
+    <link name="castor_link">
         <visual>
-            <geometry><sphere radius="0.02"/></geometry>
-            <material name="white"/>
+            <origin xyz="0 0 0" rpy="0 0 0"/>
+            <geometry>
+                <mesh filename="file://$(find final_assemble_rover_description)/meshes/castor_ball.STL" scale="1 1 1"/>
+            </geometry>
+            <material name="silver">
+                <color rgba="0.75 0.75 0.75 1.0"/>
+            </material>
         </visual>
         <collision>
-            <geometry><sphere radius="0.02"/></geometry>
+            <origin xyz="0 0 0" rpy="0 0 0"/>
+            <geometry>
+                <sphere radius="0.015"/>
+            </geometry>
         </collision>
-        <xacro:sphere_inertia m="0.1" r="0.02"/>
+        <xacro:sphere_inertia m="0.1" r="0.015"/>
     </link>
-    <gazebo reference="castor_wheel">
-        <material>Gazebo/White</material>
-        <mu1>0.0001</mu1>
-        <mu2>0.0001</mu2>
-    </gazebo>
-    <!-- TOP-MOUNTED VIRTUAL LIDAR PUCK -->
+    <!-- LIDAR LINK -->
     <joint name="lidar_joint" type="fixed">
-        <parent link="mid_deck_link"/>
+        <parent link="base_link"/>
         <child link="lidar_link"/>
-        <origin xyz="0 0 0.022" rpy="0 0 0"/>
+        <origin xyz="0 0 0.05" rpy="0 0 0"/>
     </joint>
     <link name="lidar_link">
-        <!-- Core Rotating Scanner Head -->
         <visual>
-            <geometry><cylinder radius="0.03" length="0.035"/></geometry>
+            <origin xyz="0 0 0" rpy="0 0 0"/>
+            <geometry>
+                <mesh filename="file://$(find final_assemble_rover_description)/meshes/laser_link.STL" scale="1 1 1"/>
+            </geometry>
             <material name="black"/>
         </visual>
-        <!-- Optical Sensor Lens Embellishment -->
-        <visual>
-            <origin xyz="0.025 0 0.005" rpy="0 1.5708 0"/>
-            <geometry><cylinder radius="0.006" length="0.01"/></geometry>
-            <material name="grey"/>
-        </visual>
         <collision>
-            <geometry><cylinder radius="0.03" length="0.035"/></geometry>
+            <origin xyz="0 0 0" rpy="0 0 0"/>
+            <geometry>
+                <cylinder radius="0.03" length="0.035"/>
+            </geometry>
         </collision>
         <xacro:cylinder_inertia m="0.15" r="0.03" h="0.035"/>
     </link>
-    <gazebo reference="lidar_link"><material>Gazebo/Black</material></gazebo>
-    <!-- GAZEBO KINEMATIC CONTROL PLUGIN (Differential Drive Configuration) -->
-    <gazebo>
-        <plugin name="diff_drive" filename="libgazebo_ros_diff_drive.so">
-            <ros><namespace>/</namespace></ros>
-            <left_joint>left_wheel_joint</left_joint>
-            <right_joint>right_wheel_joint</right_joint>
-            <wheel_separation>0.136</wheel_separation>
-            <wheel_diameter>0.06</wheel_diameter>
-            <max_wheel_torque>15</max_wheel_torque>
-            <max_wheel_acceleration>1.5</max_wheel_acceleration>
-            <publish_odom>true</publish_odom>
-            <publish_odom_tf>true</publish_odom_tf>
-            <publish_wheel_tf>true</publish_wheel_tf>
-            <odometry_frame>odom</odometry_frame>
-            <robot_base_frame>base_footprint</robot_base_frame>
-        </plugin>
-    </gazebo>
-    <!-- GAZEBO SENSOR PLUGIN (Virtual LiDAR Linkage for Navigation Tricking) -->
-    <gazebo reference="lidar_link">
-        <sensor type="ray" name="virtual_lidar">
-            <pose>0 0 0 0 0 0</pose>
-            <visualize>true</visualize>
-            <update_rate>10</update_rate>
-            <ray>
-                <scan>
-                    <horizontal>
-                        <samples>360</samples>
-                        <resolution>1</resolution>
-                        <min_angle>-3.14159</min_angle>
-                        <max_angle>3.14159</max_angle>
-                    </horizontal>
-                </scan>
-                <range>
-                    <min>0.12</min>
-                    <max>10.0</max>
-                    <resolution>0.01</resolution>
-                </range>
-            </ray>
-            <plugin name="scan" filename="libgazebo_ros_ray_sensor.so">
-                <ros><remapping>~/out:=scan</remapping></ros>
-                <output_type>sensor_msgs/LaserScan</output_type>
-                <frame_name>lidar_link</frame_name>
-            </plugin>
-        </sensor>
-    </gazebo>
+    <!-- GAZEBO COLOR FIXES -->
+    <gazebo reference="base_link"><material>Gazebo/Red</material></gazebo>
+    <gazebo reference="left_wheel"><material>Gazebo/Black</material></gazebo>
+    <gazebo reference="right_wheel"><material>Gazebo/Black</material></gazebo>
+    <gazebo reference="castor_link"><material>Gazebo/Silver</material></gazebo>
+    <gazebo reference="lidar_link"><material>Gazebo/DarkGrey</material></gazebo>
 </robot>
