Commit message: try

File: onshape_rover_files/robot.urdf (robot description, URDF)
Before this commit: robot onshape_rover_files, 1 links, 0 joints
Links:
- added link castor_link_1_1, mass 0.00387924; collision mesh filename=package://assets/castor_link_1_1.stl; visual mesh filename=package://assets/castor_link_1_1.stl
- added link left_wheel_link_1_1, mass 0.0327076; collision mesh filename=package://assets/left_wheel_link_1_1.stl; visual mesh filename=package://assets/left_wheel_link_1_1.stl
- added link right_wheel_link_1_1, mass 0.0327076; collision mesh filename=package://assets/right_wheel_link_1_1.stl; visual mesh filename=package://assets/right_wheel_link_1_1.stl
Joints:
- added joint castor_joint: type ball, parent base_link, child castor_link_1_1, origin xyz=0.0397465 0 -0.0076 rpy=-1.67306 -0.644916 1.42189, axis 0 0 1, limit effort=10 velocity=10
- added joint left_wheel_joint: type continuous, parent base_link, child right_wheel_link_1_1, origin xyz=-0.029 -0.05613 0.025 rpy=1.5708 -1.37617 3.14159, axis 0 0 1, limit effort=10 velocity=10
- added joint right_wheel_joint: type continuous, parent base_link, child left_wheel_link_1_1, origin xyz=-0.029 0.05613 0.025 rpy=1.5708 -0 0, axis 0 0 1, limit effort=10 velocity=10
