Commit message: update_check

File: rover_assembly_description/urdf/rover_assembly_description.urdf (robot description, URDF)
Before this commit: robot rover_assembly_description, 6 links, 5 joints
Joints:
- joint castor_joint: origin xyz=0.038053 -0.0069786 -0.033058 rpy=-0.0010351 -0.035786 -3.1416 -> xyz=0.038053 -0.0069786 -0.013058 rpy=-0.0010351 -0.035786 -3.1416; type continuous -> fixed

Commit message: trial_check

File: rover_assembly_description/urdf/rover_assembly_description.urdf (robot description, URDF)
Before this commit: robot rover_assembly_description, 6 links, 5 joints
Joints:
- joint castor_joint: origin xyz=0.038053 -0.0069786 -0.013058 rpy=-0.0010351 -0.035786 -3.1416 -> xyz=0.038053 -0.0069786 -0.026058 rpy=-0.0010351 -0.035786 -3.1416

Commit message: rover_in

File: rover_assembly_description/urdf/rover_assembly_description.urdf (robot description, URDF)
Before this commit: robot rover_assembly_description, 6 links, 5 joints
Joints:
- joint castor_joint: origin xyz=0.038053 -0.0069786 -0.026058 rpy=-0.0010351 -0.035786 -3.1416 -> xyz=0.038053 -0.0069786 -0.028058 rpy=-0.0010351 -0.035786 -3.1416

Commit message: update

File: rover_assembly_description/urdf/rover_assembly_description.urdf (robot description, URDF)
Before this commit: robot rover_assembly_description, 6 links, 5 joints
Joints:
- joint left_wheel_joint : axis 0 0 1 -> 0 0 -1

Commit message: joint

File: rover_assembly_description/urdf/rover_assembly_description.urdf (robot description, URDF)
Before this commit: robot rover_assembly_description, 6 links, 5 joints
Joints:
- removed joint left_wheel_joint 
- added joint left_wheel_joint: type continuous, parent base_link, child left_wheel_link, origin xyz=-0.030862 0.060664 0.00024787 rpy=1.5698 0 3.1407, axis 0 0 -1
